File: Notecarrier-F/KiCad_format/Notecarrier-F.kicad_sch (KiCad schematic)
At the start: 15 parts

Commit message: Merge pending library into main.
Parts:
- FID1, FID2, FID3, FID4, FID5, FID6: footprint blues-kicad-lib-pending:FIDUCIAL -> blues-kicad-lib:FIDUCIAL-F
- G1: footprint blues-kicad-lib-pending:Logo_19.5x12.5 -> blues-kicad-lib:Logo_19.5x12.5
- H1, H2, H3, H4: footprint blues-kicad-lib-pending:MountingHole_3.3mm_no-courtyard -> blues-kicad-lib:MountingHole_3.3mm_no-courtyard
- H5_1, H5_2, H5_3, H5_4: footprint blues-kicad-lib-pending:MountingHole_2.54mm_no-courtyard -> blues-kicad-lib:MountingHole_2.54mm_no-courtyard
Changed lines of the file:
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@@
       (effects (font (size 1.27 1.27)) (justify left) hide)
     )
-    (property "Footprint" "blues-kicad-lib-pending:FIDUCIAL" (at 161.29 236.22 0)
+    (property "Footprint" "blues-kicad-lib:FIDUCIAL-F" (at 161.29 236.22 0)
       (effects (font (size 1.27 1.27)) hide)
     )
@@
       (effects (font (size 1.27 1.27)) (justify left) hide)
     )
-    (property "Footprint" "blues-kicad-lib-pending:FIDUCIAL" (at 173.99 236.22 0)
+    (property "Footprint" "blues-kicad-lib:FIDUCIAL-F" (at 173.99 236.22 0)
       (effects (font (size 1.27 1.27)) hide)
     )
@@
       (effects (font (size 1.27 1.27)) (justify left) hide)
     )
-    (property "Footprint" "blues-kicad-lib-pending:MountingHole_3.3mm_no-courtyard" (at 204.47 242.57 0)
+    (property "Footprint" "blues-kicad-lib:MountingHole_3.3mm_no-courtyard" (at 204.47 242.57 0)
       (effects (font (size 1.27 1.27)) hide)
     )
@@
       (effects (font (size 1.27 1.27)) (justify left) hide)
     )
-    (property "Footprint" "blues-kicad-lib-pending:MountingHole_3.3mm_no-courtyard" (at 195.58 242.57 0)
+    (property "Footprint" "blues-kicad-lib:MountingHole_3.3mm_no-courtyard" (at 195.58 242.57 0)
       (effects (font (size 1.27 1.27)) hide)
     )
@@
       (effects (font (size 1.27 1.27)) (justify left) hide)
     )
-    (property "Footprint" "blues-kicad-lib-pending:MountingHole_2.54mm_no-courtyard" (at 224.79 236.22 0)
+    (property "Footprint" "blues-kicad-lib:MountingHole_2.54mm_no-courtyard" (at 224.79 236.22 0)
       (effects (font (size 1.27 1.27)) hide)
     )
@@
       (effects (font (size 1.27 1.27)))
     )
-    (property "Footprint" "blues-kicad-lib-pending:Logo_19.5x12.5" (at 247.65 238.76 0)
+    (property "Footprint" "blues-kicad-lib:Logo_19.5x12.5" (at 247.65 238.76 0)
       (effects (font (size 1.27 1.27)) hide)
     )
@@
       (effects (font (size 1.27 1.27)) (justify left) hide)
     )
-    (property "Footprint" "blues-kicad-lib-pending:MountingHole_2.54mm_no-courtyard" (at 214.63 242.57 0)
+    (property "Footprint" "blues-kicad-lib:MountingHole_2.54mm_no-courtyard" (at 214.63 242.57 0)
       (effects (font (size 1.27 1.27)) hide)
     )
@@
       (effects (font (size 1.27 1.27)) (justify left) hide)
     )
-    (property "Footprint" "blues-kicad-lib-pending:MountingHole_3.3mm_no-courtyard" (at 195.58 236.22 0)
+    (property "Footprint" "blues-kicad-lib:MountingHole_3.3mm_no-courtyard" (at 195.58 236.22 0)
       (effects (font (size 1.27 1.27)) hide)
     )
@@
       (effects (font (size 1.27 1.27)) (justify left) hide)
     )
-    (property "Footprint" "blues-kicad-lib-pending:FIDUCIAL" (at 173.99 243.84 0)
+    (property "Footprint" "blues-kicad-lib:FIDUCIAL-F" (at 173.99 243.84 0)
       (effects (font (size 1.27 1.27)) hide)
     )
@@
       (effects (font (size 1.27 1.27)) (justify left) hide)
     )
-    (property "Footprint" "blues-kicad-lib-pending:FIDUCIAL" (at 161.29 240.03 0)
+    (property "Footprint" "blues-kicad-lib:FIDUCIAL-F" (at 161.29 240.03 0)
       (effects (font (size 1.27 1.27)) hide)
     )
@@
       (effects (font (size 1.27 1.27)) (justify left) hide)
     )
-    (property "Footprint" "blues-kicad-lib-pending:MountingHole_2.54mm_no-courtyard" (at 214.63 236.22 0)
+    (property "Footprint" "blues-kicad-lib:MountingHole_2.54mm_no-courtyard" (at 214.63 236.22 0)
       (effects (font (size 1.27 1.27)) hide)
     )
@@
       (effects (font (size 1.27 1.27)) (justify left) hide)
     )
-    (property "Footprint" "blues-kicad-lib-pending:FIDUCIAL" (at 173.99 240.03 0)
+    (property "Footprint" "blues-kicad-lib:FIDUCIAL-F" (at 173.99 240.03 0)
       (effects (font (size 1.27 1.27)) hide)
     )
@@
       (effects (font (size 1.27 1.27)) (justify left) hide)
     )
-    (property "Footprint" "blues-kicad-lib-pending:FIDUCIAL" (at 161.29 243.84 0)
+    (property "Footprint" "blues-kicad-lib:FIDUCIAL-F" (at 161.29 243.84 0)
       (effects (font (size 1.27 1.27)) hide)
     )
@@
       (effects (font (size 1.27 1.27)) (justify left) hide)
     )
-    (property "Footprint" "blues-kicad-lib-pending:MountingHole_2.54mm_no-courtyard" (at 224.79 242.57 0)
+    (property "Footprint" "blues-kicad-lib:MountingHole_2.54mm_no-courtyard" (at 224.79 242.57 0)
       (effects (font (size 1.27 1.27)) hide)
     )
@@
       (effects (font (size 1.27 1.27)) (justify left) hide)
     )
-    (property "Footprint" "blues-kicad-lib-pending:MountingHole_3.3mm_no-courtyard" (at 204.47 236.22 0)
-      (effects (font (size 1.27 1.27)) hide)
-    )
+    (property "Footprint" "blues-kicad-lib:MountingHole_3.3mm_no-courtyard" (at 204.47 236.22 0)
+      (effects (font (size 1.27 1.27)) hide)
+    )
