File: Notecarrier-F/KiCad_format/Notecarrier-F_Notecard.kicad_sch (KiCad schematic)
At the start: 0 parts

Commit message: Port Notecarrier-F schematic and BOM.
Parts:
- added C3 (x2): 0.1µF, symbol Device:C
- added C3 (x3): 33pF, symbol Device:C
- added F1: F1.5A, symbol Device:Fuse
- added F2: 3.5A/32V, symbol Device:Fuse
- added J5: NanoSIM - SF72S006VBAR2500, Connector_JAE:JAE_SIM_Card_SF72S006, symbol blues-kicad-lib:SF72S006VBDR2500
- added J6: MDT420E01001, blues-kicad-lib:J-75-0050-MOS-M2-E, symbol blues-kicad-lib:MDT420E01001
- added OBJ1: 9774025151R, blues-kicad-lib:9774025151R, symbol blues-kicad-lib:RND_STNDFF_M2.5X0.45_STEEL_2.5MM
- added R16: 15k, symbol Device:R
- added R3: 10kOhms, symbol Device:R
- added R5 (x3): 22R, symbol Device:R
- added RR1, RR2: 741X163101JP, symbol blues-kicad-lib:R_Array08
- added SW1: CJS-1200TA, blues-kicad-lib:CJS-1200TA, symbol blues-kicad-lib:CJS-1200TA
- added SW2: PTS810SJK250SMTRLFS, symbol Switch:SW_Push
- added TVS2: PESD5V0L5UV, Package_TO_SOT_SMD:SOT-666, symbol blues-kicad-lib:PESD5V0L5UV
Connections:
- new net: C3.1, J5.C3 (CLK), R5.1, TVS2.1 (K1)
- new net: C3.1, J5.C7 (I/O), R16.2, R5.1, TVS2.6 (K5)
- new net: C3.1, J5.C2 (RST), R5.1, TVS2.5 (K4)
- new net: F2.2, J6.70 (VMODEM_P), J6.72 (VMODEM_P), J6.74 (VMODEM_P)
- new net: J6.20 (VACT_GPS_OUT), SW1.2 (B)
- new net: J6.22 (VACT_GPS_IN), SW1.1 (C)
- new net: J6.40 (SCL_P), RR2.16 (R1_2)
- new net: J6.42 (SDA_P), RR2.15 (R2_2)
- new net: RR1.10 (R7_2), RR2.7 (R7_1)
- new net: RR1.11 (R6_2), RR2.6 (R6_1)
- new net: RR1.12 (R5_2), RR2.5 (R5_1)
- new net: RR1.13 (R4_2), RR2.4 (R4_1)
- new net: RR1.14 (R3_2), RR2.3 (R3_1)
- new net: RR1.15 (R2_2), RR2.2 (R2_1)
- new net: RR1.16 (R1_2), RR2.1 (R1_1)
- new net: RR1.9 (R8_2), RR2.8 (R8_1)
- new net ATTN_P: J6.54 (ATTN_P), RR2.14 (R3_2)
- new net AUX_EN_P: J6.56 (AUX_EN_P), RR2.13 (R4_2)
- new net AUX_RX_P: J6.58 (AUX_RX_P), RR2.12 (R5_2)
- new net AUX_TX_P: J6.60 (AUX_TX_P), RR2.11 (R6_2)
- new net D_N: J6.9 (USB_DM)
- new net D_P: J6.7 (USB_DP)
- new net GND: C3.2, C3.2, C3.2, C3.2, C3.2, J5.C5 (GND), J5.CSW, J5.SH, J6.11 (GND), J6.18 (GND), J6.3 (GND), J6.33 (GND), J6.39 (GND), J6.45 (GND), J6.5 (GND), J6.51 (GND), J6.57 (GND), J6.6 (GND), J6.71 (GND), J6.73 (GND), SW2.2, TVS2.2 (A)
- new net N_ATTN: RR1.3 (R3_1)
- new net N_AUX1: J6.46 (AUX1)
- new net N_AUX2: J6.48 (AUX2)
- new net N_AUX3: J6.50 (AUX3)
- new net N_AUX4: J6.52 (AUX4)
- new net N_AUX5: J6.38 (NC38)
- new net N_AUX_EN: RR1.4 (R4_1)
- new net N_AUX_RX: RR1.5 (R5_1)
- new net N_AUX_TX: RR1.6 (R6_1)
- new net N_NRST: C3.1, J6.67 (NRST), R3.2, SW2.1
- new net N_RX: RR1.7 (R7_1)
- new net N_SCL: RR1.1 (R1_1)
- new net N_SDA: RR1.2 (R2_1)
- new net N_TX: RR1.8 (R8_1)
- new net N_VIO: F1.1, R3.1
- new net RX_P: J6.62 (RX_P), RR2.10 (R7_2)
- new net SIM_CLK: J6.14 (SIM_CLK), R5.2
- new net SIM_IO: J6.12 (SIM_IO), R5.2
- new net SIM_NPRESENT: J5.DSW, J6.16 (SIM_NPRESENT), TVS2.4 (K3)
- new net SIM_RST: J6.10 (SIM_RST), R5.2
- new net SIM_VCC: C3.1, J5.C1 (VCC), J6.8 (SIM_VCC), R16.1, TVS2.3 (K2)
- new net TX_P: J6.64 (TX_P), RR2.9 (R8_2)
- new net VIO_P: F1.2, J6.2 (VIO_P), J6.4 (VIO_P)
- new net VMAIN: F2.1
- new net VUSB: J6.13 (VUSB)
- no-connect marks 0 -> 29
Other:
- note added: "ACTIVE"
- note added: "Label Promotion"
- note added: "Notecard Connector"
- note added: "One of the net labels on this sheet need to be common with other sheets. In the original Altium source files, this was achieved for some labels by adding Off-Sheet Connectors to the nets. But the remainder (inadvertently perhaps) rely on promoting all net labels to global using the "Net Identifier Scope" setting. This renders the original Off Sheet Connectors redundant. To avoid losing that disti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"
- note added: "PASSIVE"
- note added: "RESET"
- note added: "SIM Card"
- title: (none) -> Notecarrier-F

Commit message: Ported footprint assignments, board outline, copper layers and dimensional drawings for Notecarrier-F.
Footprints currently held in a “blues-kicad-lib-pending” library, prior to merging with “blues-kicad-lib” and deleting unused items.
Parts:
- C3: footprint (none) -> blues-kicad-lib-pending:CAP 0402_1005
- F1, F2: footprint (none) -> blues-kicad-lib:FS-0603
- J5: footprint Connector_JAE:JAE_SIM_Card_SF72S006 -> blues-kicad-lib-pending:J-NANOSIM-SF72S006VBA
- J6: footprint blues-kicad-lib:J-75-0050-MOS-M2-E -> blues-kicad-lib-pending:J-75-0050-MOS-M2
- OBJ1: footprint blues-kicad-lib:9774025151R -> blues-kicad-lib:DIST-WASMSIM0250
- R16, R3, R5: footprint (none) -> blues-kicad-lib-pending:RES 0402_1005
- RR1, RR2: footprint (none) -> blues-kicad-lib-pending:RESNET 1506-16 CONVEX
- SW1: footprint blues-kicad-lib:CJS-1200TA -> blues-kicad-lib-pending:SW_CJS-1200TA
- SW2: footprint (none) -> blues-kicad-lib-pending:C&K PTS810
- TVS2: footprint Package_TO_SOT_SMD:SOT-666 -> blues-kicad-lib-pending:SOT666
Changed lines of the file:
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@@
       (effects (font (size 1.27 1.27)) (justify left))
     )
-    (property "Footprint" "" (at 301.9552 114.3 0)
+    (property "Footprint" "blues-kicad-lib-pending:CAP 0402_1005" (at 301.9552 114.3 0)
       (effects (font (size 1.27 1.27)) hide)
     )
@@
       (effects (font (size 1.27 1.27)) (justify left))
     )
-    (property "Footprint" "" (at 312.1152 114.3 0)
+    (property "Footprint" "blues-kicad-lib-pending:CAP 0402_1005" (at 312.1152 114.3 0)
       (effects (font (size 1.27 1.27)) hide)
     )
@@
       (effects (font (size 1.27 1.27)))
     )
-    (property "Footprint" "" (at 205.74 187.96 0)
+    (property "Footprint" "blues-kicad-lib-pending:C&K PTS810" (at 205.74 187.96 0)
       (effects (font (size 1.27 1.27)) hide)
     )
@@
       (effects (font (size 1.27 1.27)) (justify left))
     )
-    (property "Footprint" "" (at 317.1952 114.3 0)
+    (property "Footprint" "blues-kicad-lib-pending:CAP 0402_1005" (at 317.1952 114.3 0)
       (effects (font (size 1.27 1.27)) hide)
     )
@@
       (effects (font (size 1.27 1.27)) (justify left))
     )
-    (property "Footprint" "" (at 181.3052 209.55 0)
+    (property "Footprint" "blues-kicad-lib-pending:CAP 0402_1005" (at 181.3052 209.55 0)
       (effects (font (size 1.27 1.27)) hide)
     )
@@
       (effects (font (size 1.27 1.27)) (justify left))
     )
-    (property "Footprint" "" (at 278.13 68.072 90)
+    (property "Footprint" "blues-kicad-lib-pending:RES 0402_1005" (at 278.13 68.072 90)
       (effects (font (size 1.27 1.27)) hide)
     )
@@
       (effects (font (size 1.27 1.27)) (justify right))
     )
-    (property "Footprint" "" (at 93.98 204.978 90)
+    (property "Footprint" "blues-kicad-lib:FS-0603" (at 93.98 204.978 90)
       (effects (font (size 1.27 1.27)) hide)
     )
@@
       (effects (font (size 1.27 1.27)) (justify left))
     )
-    (property "Footprint" "" (at 278.13 70.612 90)
+    (property "Footprint" "blues-kicad-lib-pending:RES 0402_1005" (at 278.13 70.612 90)
       (effects (font (size 1.27 1.27)) hide)
     )
@@
       (effects (font (size 1.27 1.27)))
     )
-    (property "Footprint" "blues-kicad-lib:9774025151R" (at 86.36 101.6 0)
+    (property "Footprint" "blues-kicad-lib:DIST-WASMSIM0250" (at 86.36 101.6 0)
       (effects (font (size 1.27 1.27)) hide)
     )
@@
       (effects (font (size 1.27 1.27)))
     )
-    (property "Footprint" "blues-kicad-lib:J-75-0050-MOS-M2-E" (at 137.16 210.82 0)
+    (property "Footprint" "blues-kicad-lib-pending:J-75-0050-MOS-M2" (at 137.16 210.82 0)
       (effects (font (size 1.27 1.27)) hide)
     )
@@
       (effects (font (size 1.27 1.27)) (justify left))
     )
-    (property "Footprint" "" (at 307.0352 114.3 0)
+    (property "Footprint" "blues-kicad-lib-pending:CAP 0402_1005" (at 307.0352 114.3 0)
       (effects (font (size 1.27 1.27)) hide)
     )
@@
       (effects (font (size 1.27 1.27)) (justify left))
     )
-    (property "Footprint" "Connector_JAE:JAE_SIM_Card_SF72S006" (at 361.95 106.68 0)
+    (property "Footprint" "blues-kicad-lib-pending:J-NANOSIM-SF72S006VBA" (at 361.95 106.68 0)
       (effects (font (size 1.27 1.27)) hide)
     )
@@
       (effects (font (size 1.27 1.27)) (justify right))
     )
-    (property "Footprint" "" (at 85.09 114.808 90)
+    (property "Footprint" "blues-kicad-lib:FS-0603" (at 85.09 114.808 90)
       (effects (font (size 1.27 1.27)) hide)
     )
@@
       (effects (font (size 1.27 1.27)) (justify left))
     )
-    (property "Footprint" "" (at 291.592 59.69 90)
+    (property "Footprint" "blues-kicad-lib-pending:RES 0402_1005" (at 291.592 59.69 90)
       (effects (font (size 1.27 1.27)) hide)
     )
@@
       (effects (font (size 1.27 1.27)) (justify left))
     )
-    (property "Footprint" "" (at 278.13 80.772 90)
+    (property "Footprint" "blues-kicad-lib-pending:RES 0402_1005" (at 278.13 80.772 90)
       (effects (font (size 1.27 1.27)) hide)
     )
@@
       (effects (font (size 1.27 1.27)) (justify left))
     )
-    (property "Footprint" "" (at 187.452 182.88 90)
+    (property "Footprint" "blues-kicad-lib-pending:RES 0402_1005" (at 187.452 182.88 90)
       (effects (font (size 1.27 1.27)) hide)
     )
@@
       (effects (font (size 1.27 1.27)))
     )
-    (property "Footprint" "" (at 52.07 195.834 0)
+    (property "Footprint" "blues-kicad-lib-pending:RESNET 1506-16 CONVEX" (at 52.07 195.834 0)
       (effects (font (size 1.27 1.27)) hide)
     )
@@
       (effects (font (size 1.27 1.27)) (justify right))
     )
-    (property "Footprint" "Package_TO_SOT_SMD:SOT-666" (at 336.55 123.19 0)
+    (property "Footprint" "blues-kicad-lib-pending:SOT666" (at 336.55 123.19 0)
       (effects (font (size 1.27 1.27)) hide)
     )
@@
       (effects (font (size 1.27 1.27)))
     )
-    (property "Footprint" "" (at 71.12 195.834 0)
+    (property "Footprint" "blues-kicad-lib-pending:RESNET 1506-16 CONVEX" (at 71.12 195.834 0)
       (effects (font (size 1.27 1.27)) hide)
     )
@@
       (effects (font (size 1.27 1.27)))
     )
-    (property "Footprint" "blues-kicad-lib:CJS-1200TA" (at 73.66 143.51 0)
-      (effects (font (size 1.27 1.27)) hide)
-    )
+    (property "Footprint" "blues-kicad-lib-pending:SW_CJS-1200TA" (at 73.66 143.51 0)
+      (effects (font (size 1.27 1.27)) hide)
+    )
