File: Notecarrier-F/KiCad_format/Notecarrier-F_Power.kicad_sch (KiCad schematic)
At the start: 48 parts, among them J1 S2BPHSM4TBLFSN, J2 S2BPHSM4TBLFSN, J3 S2BPHSM4TBLFSN, J4 10118193-0001LF, U1 TPS62748YFPT, U2 BQ24210DQCT, U3 TPS63020DSJR, U5 MAX17225ELT+

Commit message: Merge pending library into main.
Parts:
- C1, C4: footprint blues-kicad-lib-pending:CAP 1206_3216 - 0.8MM -> blues-kicad-lib:CAP 1206_3216 - 0.8MM
- C10, C11, C14, C15, C18, C19, C2, C20, C21, C25, C3: footprint blues-kicad-lib-pending:CAP 0402_1005 -> blues-kicad-lib:CAP 0402_1005
- C12: footprint blues-kicad-lib-pending:CAP 1210_3225 - 2.8MM -> blues-kicad-lib:CAP 1210_3225 - 2.8MM
- C13, C16, C17: footprint blues-kicad-lib-pending:CAP 0603_1608 -> blues-kicad-lib:CAP 0603_1608
- C22, C23, C24: footprint blues-kicad-lib-pending:CAP FILM 0805 -> blues-kicad-lib:CAP FILM 0805
- DS3, DS6, DS7: footprint blues-kicad-lib-pending:DO214AA SMB -> blues-kicad-lib:DO214AA SMB
- J1, J2, J3: footprint blues-kicad-lib-pending:JST S2B-PH-SM4-TB -> blues-kicad-lib:JST S2B-PH-SM4-TB
- J4: footprint blues-kicad-lib-pending:FCI USB 10118193-0001LF -> blues-kicad-lib:FCI USB 10118193-0001LF
- L1: footprint blues-kicad-lib-pending:IND_XFL4020-222MEC -> blues-kicad-lib:IND_XFL4020-222MEC
- L2: footprint blues-kicad-lib-pending:VCHA042A-1R5MS6 -> blues-kicad-lib:VCHA042A-1R5MS6
- L3: footprint blues-kicad-lib-pending:1285AS-H-2R2M=P2-INDC2016X100N -> blues-kicad-lib:1285AS-H-2R2M=P2-INDC2016X100N
- R1, R13, R14, R16, R17, R2, R3, R4: footprint blues-kicad-lib-pending:RES 0402_1005 -> blues-kicad-lib:RES 0402_1005
- R5: footprint blues-kicad-lib-pending:RES 1206_3216 -> blues-kicad-lib:RES 1206_3216
- TVS1: footprint blues-kicad-lib-pending:SMB_Backwards -> blues-kicad-lib:SMB_Backwards
- U1: footprint blues-kicad-lib-pending:TPS62748YFPT-DSBGA4x2 -> blues-kicad-lib:TPS62748YFPT-DSBGA4x2
- U3: footprint blues-kicad-lib-pending:TI PVSON-14 DSJ -> blues-kicad-lib:TI PVSON-14 DSJ
- U5: footprint blues-kicad-lib-pending:MAX17225ELT+UDFN -> blues-kicad-lib:MAX17225ELT+UDFN
