File: Notecarrier-B/KiCad_format/Notecarrier-B.kicad_pcb (KiCad board)
At the start: 2 copper layers, 51.1 x 45.6 mm, 96 parts, among them J19 MICROUSB-B, J20 MDT420E01001, J21 NU, J22 NU, J23 S2B-PH-SM4-TB(LF)(SN), J24 SM04B-SRSS-TBT, Q2 AO3420, U3 MAX17225ELT, U4 TPS62748YFPT, U5 MCP73831-2ACI/MC

Commit message: Backport SOT23 footprint name change from Notecarrier-A.
Parts:
- Q2: footprint blues-kicad-lib:SOT23 -> blues-kicad-lib:SOT23_NO-FILL
Changed lines of the file:
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@@
   (net 84 "Net-(RR1-R1.2)")
   (net 85 "unconnected-(U5-NC-Pad7)")
-  (net 86 "Net-(#PWR037-USB_SHIELD)")
-  (net 87 "Net-(#FLG08-pwr)")
+  (net 86 "Net-(J19-Shield)")
+  (net 87 "Net-(J20-VACT_GPS_IN)")
   (footprint "blues-kicad-lib:J-75-0050-MOS-M2-E" (layer "F.Cu")
     (at 102.46 77.14 90)
@@
       (net 33 "unconnected-(J20-NC21-Pad21)") (pinfunction "NC21") (pintype "passive+no_connect") (solder_mask_margin 0.05) (zone_connect 0))
     (pad "22" smd rect (at -4 2.275 90) (size 0.3 1.55) (layers "F.Cu" "F.Paste" "F.Mask")
-      (net 87 "Net-(#FLG08-pwr)") (pinfunction "VACT_GPS_IN") (pintype "power_in") (solder_mask_margin 0.05) (zone_connect 0))
+      (net 87 "Net-(J20-VACT_GPS_IN)") (pinfunction "VACT_GPS_IN") (pintype "power_in") (solder_mask_margin 0.05) (zone_connect 0))
     (pad "23" smd rect (at -3.75 -5.275 90) (size 0.3 1.55) (layers "F.Cu" "F.Paste" "F.Mask")
       (net 34 "unconnected-(J20-NC23-Pad23)") (pinfunction "NC23") (pintype "passive+no_connect") (solder_mask_margin 0.05) (zone_connect 0))
@@
       (net 2 "GND") (pinfunction "GND") (pintype "power_out") (solder_mask_margin 0.05))
     (pad "6" smd rect (at -3.8 2.55 90) (size 1.8 1.9) (layers "F.Cu" "F.Paste" "F.Mask")
-      (net 86 "Net-(#PWR037-USB_SHIELD)") (pinfunction "Shield") (pintype "passive") (solder_mask_margin 0.05))
+      (net 86 "Net-(J19-Shield)") (pinfunction "Shield") (pintype "passive") (solder_mask_margin 0.05))
     (pad "6" smd rect (at -3.05 0 90) (size 2.1 1.6) (layers "F.Cu" "F.Paste" "F.Mask")
-      (net 86 "Net-(#PWR037-USB_SHIELD)") (pinfunction "Shield") (pintype "passive") (solder_mask_margin 0.05))
+      (net 86 "Net-(J19-Shield)") (pinfunction "Shield") (pintype "passive") (solder_mask_margin 0.05))
     (pad "6" smd rect (at -1.2 2.55 90) (size 1.9 1.9) (layers "F.Cu" "F.Paste" "F.Mask")
-      (net 86 "Net-(#PWR037-USB_SHIELD)") (pinfunction "Shield") (pintype "passive") (solder_mask_margin 0.05))
+      (net 86 "Net-(J19-Shield)") (pinfunction "Shield") (pintype "passive") (solder_mask_margin 0.05))
     (pad "6" smd rect (at 1.2 2.55 90) (size 1.9 1.9) (layers "F.Cu" "F.Paste" "F.Mask")
-      (net 86 "Net-(#PWR037-USB_SHIELD)") (pinfunction "Shield") (pintype "passive") (solder_mask_margin 0.05))
+      (net 86 "Net-(J19-Shield)") (pinfunction "Shield") (pintype "passive") (solder_mask_margin 0.05))
     (pad "6" smd rect (at 3.05 0 90) (size 2.1 1.6) (layers "F.Cu" "F.Paste" "F.Mask")
-      (net 86 "Net-(#PWR037-USB_SHIELD)") (pinfunction "Shield") (pintype "passive") (solder_mask_margin 0.05))
+      (net 86 "Net-(J19-Shield)") (pinfunction "Shield") (pintype "passive") (solder_mask_margin 0.05))
     (pad "6" smd rect (at 3.8 2.55 90) (size 1.8 1.9) (layers "F.Cu" "F.Paste" "F.Mask")
-      (net 86 "Net-(#PWR037-USB_SHIELD)") (pinfunction "Shield") (pintype "passive") (solder_mask_margin 0.05))
+      (net 86 "Net-(J19-Shield)") (pinfunction "Shield") (pintype "passive") (solder_mask_margin 0.05))
     (model "${BLUES_KICAD_LIB_DIR}/3d-models/J-5-0065-FOS-MICROUSB10118192.step"
       (offset (xyz 0 0 0))
@@
       (stroke (width 0.2) (type solid)) (layer "B.Fab"))
     (pad "1" smd rect (at -1.5 0 90) (size 1.15 1.8) (layers "B.Cu" "B.Paste" "B.Mask")
-      (net 86 "Net-(#PWR037-USB_SHIELD)") (pintype "passive") (solder_mask_margin 0.1))
+      (net 86 "Net-(J19-Shield)") (pintype "passive") (solder_mask_margin 0.1))
     (pad "2" smd rect (at 1.4 0 90) (size 1.15 1.8) (layers "B.Cu" "B.Paste" "B.Mask")
       (net 2 "GND") (pintype "passive") (solder_mask_margin 0.1))
@@
       (stroke (width 0.2) (type solid)) (layer "B.Fab"))
     (pad "1" smd rect (at 0 3.81 180) (size 1 1.27) (layers "B.Cu" "B.Paste" "B.Mask")
-      (net 87 "Net-(#FLG08-pwr)") (pintype "passive") (solder_mask_margin 0.1))
+      (net 87 "Net-(J20-VACT_GPS_IN)") (pintype "passive") (solder_mask_margin 0.1))
     (pad "2" smd rect (at 0 -3.81 180) (size 1 1.27) (layers "B.Cu" "B.Paste" "B.Mask")
       (net 20 "VACT_GPS_OUT") (pintype "passive") (solder_mask_margin 0.1))
@@
     )
   )
-  (footprint "blues-kicad-lib:SOT23" (layer "B.Cu")
+  (footprint "blues-kicad-lib:SOT23_NO-FILL" (layer "B.Cu")
     (at 123.31 68.24)
     (descr "SOT-23, ported from OrCad")
+    (property "Critical" "")
     (property "Description" "TRANSISTOR MOSFET N AO3420 SOT-23 ALPHA-OMEGA SMT")
+    (property "Manufacturer" "")
+    (property "Order Code" "")
+    (property "Part Number" "")
     (property "Pkg Type" "SMD")
     (property "Sheetfile" "Notecarrier-B.kicad_sch")
     (property "Sheetname" "")
+    (property "Supplier" "")
     (property "Temperature" "-55°..+150°")
     (property "ki_description" "MOSFET N-CH 20V 6A SOT23-3L")
     (property "ki_keywords" "N-Channel MOSFET")
+    (zone_connect 0)
     (attr smd)
     (fp_text reference "Q2" (at -1.1 3.2 180) (layer "B.SilkS") hide
@@
       (stroke (width 0.2) (type solid)) (layer "B.Fab"))
     (pad "1" smd rect (at 0 0) (size 0.9 0.8) (layers "B.Cu" "B.Paste" "B.Mask")
-      (net 8 "/RST") (pinfunction "G") (pintype "input") (solder_mask_margin 0.05) (zone_connect 0))
+      (net 8 "/RST") (pinfunction "G") (pintype "input") (solder_mask_margin 0.05))
     (pad "2" smd rect (at 0 1.9) (size 0.9 0.8) (layers "B.Cu" "B.Paste" "B.Mask")
-      (net 2 "GND") (pinfunction "S") (pintype "passive") (solder_mask_margin 0.05) (zone_connect 0))
+      (net 2 "GND") (pinfunction "S") (pintype "passive") (solder_mask_margin 0.05))
     (pad "3" smd rect (at -2.37 0.95) (size 0.9 0.8) (layers "B.Cu" "B.Paste" "B.Mask")
-      (net 57 "/NRST") (pinfunction "D") (pintype "passive") (solder_mask_margin 0.05) (zone_connect 0))
+      (net 57 "/NRST") (pinfunction "D") (pintype "passive") (solder_mask_margin 0.05))
     (model "${BLUES_KICAD_LIB_DIR}/3d-models/SOT23.step"
       (offset (xyz 0 0 0))
@@
       (stroke (width 0.2) (type solid)) (layer "B.Fab"))
     (pad "1" smd rect (at -1.5 0 90) (size 0.9 1.9) (layers "B.Cu" "B.Paste" "B.Mask")
-      (net 86 "Net-(#PWR037-USB_SHIELD)") (pintype "passive") (solder_mask_margin 0.1))
+      (net 86 "Net-(J19-Shield)") (pintype "passive") (solder_mask_margin 0.1))
     (pad "2" smd rect (at 1.5 0 90) (size 0.9 1.9) (layers "B.Cu" "B.Paste" "B.Mask")
       (net 2 "GND") (pintype "passive") (solder_mask_margin 0.1))
