File: Notecarrier-B/KiCad_format/Notecarrier-B.kicad_sch (KiCad schematic)
At the start: 66 parts, among them J19 MICROUSB-B, J20 MDT420E01001, J21 NU, J22 NU, J23 S2B-PH-SM4-TB(LF)(SN), J24 SM04B-SRSS-TBT, Q2 AO3420, U3 MAX17225ELT, U4 TPS62748YFPT, U5 MCP73831-2ACI/MC

Commit message: Backport name change from `RS-0402` to `RS-0402_NO-FILL`.
Name changed in Notecarrier-A port. See those PortingNotes for details. Also performed long overdue “update PCB from schematic” - remember that the test points are not in the schematic, so must be preserved in the PCB! The update has no material effect, only updates to library references. Confirmed by comparing Gerbers before and after - only change is the fiducial mask layer has slightly smaller radius. The difference is not significant.
Parts:
- C10, C111, C115, C116, C14, C7, C8, C9: footprint blues-kicad-lib:CS-C-0402 -> blues-kicad-lib:CS-C-0402_NO-FILL
- R10, R318, R319, R322, R323, R324, R325, R326, R6: footprint blues-kicad-lib:RS-0402 -> blues-kicad-lib:RS-0402_NO-FILL
- R5, R7: footprint blues-kicad-lib:RS-0201 -> blues-kicad-lib:RS-0201_NO-FILL
Changed lines of the file:
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@@
       (effects (font (size 1.27 1.27)) (justify left))
     )
-    (property "Footprint" "blues-kicad-lib:RS-0402" (at 290.83 58.42 0)
+    (property "Footprint" "blues-kicad-lib:RS-0402_NO-FILL" (at 290.83 58.42 0)
       (effects (font (size 1.27 1.27)) hide)
     )
@@
       (effects (font (size 1.27 1.27)) (justify left))
     )
-    (property "Footprint" "blues-kicad-lib:CS-C-0402" (at 322.58 73.66 0)
+    (property "Footprint" "blues-kicad-lib:CS-C-0402_NO-FILL" (at 322.58 73.66 0)
       (effects (font (size 1.27 1.27)) hide)
     )
@@
       (effects (font (size 1.27 1.27)) (justify left))
     )
-    (property "Footprint" "blues-kicad-lib:CS-C-0402" (at 167.64 167.64 0)
+    (property "Footprint" "blues-kicad-lib:CS-C-0402_NO-FILL" (at 167.64 167.64 0)
       (effects (font (size 1.27 1.27)) hide)
     )
@@
       (effects (font (size 1.27 1.27)) (justify left))
     )
-    (property "Footprint" "blues-kicad-lib:RS-0402" (at 372.11 72.39 0)
+    (property "Footprint" "blues-kicad-lib:RS-0402_NO-FILL" (at 372.11 72.39 0)
       (effects (font (size 1.27 1.27)) hide)
     )
@@
       (effects (font (size 1.27 1.27)) (justify left))
     )
-    (property "Footprint" "blues-kicad-lib:CS-C-0402" (at 233.68 76.2 0)
+    (property "Footprint" "blues-kicad-lib:CS-C-0402_NO-FILL" (at 233.68 76.2 0)
       (effects (font (size 1.27 1.27)) hide)
     )
@@
       (effects (font (size 1.27 1.27)) (justify left))
     )
-    (property "Footprint" "blues-kicad-lib:RS-0201" (at 347.98 142.24 0)
+    (property "Footprint" "blues-kicad-lib:RS-0201_NO-FILL" (at 347.98 142.24 0)
       (effects (font (size 1.27 1.27)) hide)
     )
@@
       (effects (font (size 1.27 1.27)) (justify left))
     )
-    (property "Footprint" "blues-kicad-lib:RS-0402" (at 158.75 247.65 0)
+    (property "Footprint" "blues-kicad-lib:RS-0402_NO-FILL" (at 158.75 247.65 0)
       (effects (font (size 1.27 1.27)) hide)
     )
@@
       (effects (font (size 1.27 1.27)) (justify left))
     )
-    (property "Footprint" "blues-kicad-lib:CS-C-0402" (at 280.67 76.2 0)
+    (property "Footprint" "blues-kicad-lib:CS-C-0402_NO-FILL" (at 280.67 76.2 0)
       (effects (font (size 1.27 1.27)) hide)
     )
@@
       (effects (font (size 1.27 1.27)) (justify left))
     )
-    (property "Footprint" "blues-kicad-lib:CS-C-0402" (at 378.46 73.66 0)
+    (property "Footprint" "blues-kicad-lib:CS-C-0402_NO-FILL" (at 378.46 73.66 0)
       (effects (font (size 1.27 1.27)) hide)
     )
@@
       (effects (font (size 1.27 1.27)) (justify left))
     )
-    (property "Footprint" "blues-kicad-lib:RS-0402" (at 300.99 99.06 0)
+    (property "Footprint" "blues-kicad-lib:RS-0402_NO-FILL" (at 300.99 99.06 0)
       (effects (font (size 1.27 1.27)) hide)
     )
@@
       (effects (font (size 1.27 1.27)) (justify left))
     )
-    (property "Footprint" "blues-kicad-lib:RS-0402" (at 364.49 50.8 0)
+    (property "Footprint" "blues-kicad-lib:RS-0402_NO-FILL" (at 364.49 50.8 0)
       (effects (font (size 1.27 1.27)) hide)
     )
@@
       (effects (font (size 1.27 1.27)) (justify left))
     )
-    (property "Footprint" "blues-kicad-lib:CS-C-0402" (at 163.83 248.92 0)
+    (property "Footprint" "blues-kicad-lib:CS-C-0402_NO-FILL" (at 163.83 248.92 0)
       (effects (font (size 1.27 1.27)) hide)
     )
@@
       (effects (font (size 1.27 1.27)) (justify left))
     )
-    (property "Footprint" "blues-kicad-lib:RS-0201" (at 342.9 166.37 0)
+    (property "Footprint" "blues-kicad-lib:RS-0201_NO-FILL" (at 342.9 166.37 0)
       (effects (font (size 1.27 1.27)) hide)
     )
@@
       (effects (font (size 1.27 1.27)) (justify left))
     )
-    (property "Footprint" "blues-kicad-lib:RS-0402" (at 364.49 48.26 0)
+    (property "Footprint" "blues-kicad-lib:RS-0402_NO-FILL" (at 364.49 48.26 0)
       (effects (font (size 1.27 1.27)) hide)
     )
@@
       (effects (font (size 1.27 1.27)) (justify left))
     )
-    (property "Footprint" "blues-kicad-lib:CS-C-0402" (at 325.12 73.66 0)
+    (property "Footprint" "blues-kicad-lib:CS-C-0402_NO-FILL" (at 325.12 73.66 0)
       (effects (font (size 1.27 1.27)) hide)
     )
@@
       (effects (font (size 1.27 1.27)) (justify left))
     )
-    (property "Footprint" "blues-kicad-lib:RS-0402" (at 300.99 104.14 0)
+    (property "Footprint" "blues-kicad-lib:RS-0402_NO-FILL" (at 300.99 104.14 0)
       (effects (font (size 1.27 1.27)) hide)
     )
@@
       (effects (font (size 1.27 1.27)) (justify left))
     )
-    (property "Footprint" "blues-kicad-lib:RS-0402" (at 276.86 74.93 0)
+    (property "Footprint" "blues-kicad-lib:RS-0402_NO-FILL" (at 276.86 74.93 0)
       (effects (font (size 1.27 1.27)) hide)
     )
@@
       (effects (font (size 1.27 1.27)) (justify left))
     )
-    (property "Footprint" "blues-kicad-lib:RS-0402" (at 299.72 45.72 0)
+    (property "Footprint" "blues-kicad-lib:RS-0402_NO-FILL" (at 299.72 45.72 0)
       (effects (font (size 1.27 1.27)) hide)
     )
@@
       (effects (font (size 1.27 1.27)) (justify left))
     )
-    (property "Footprint" "blues-kicad-lib:CS-C-0402" (at 375.92 73.66 0)
-      (effects (font (size 1.27 1.27)) hide)
-    )
+    (property "Footprint" "blues-kicad-lib:CS-C-0402_NO-FILL" (at 375.92 73.66 0)
+      (effects (font (size 1.27 1.27)) hide)
+    )

Commit message: Backport SOT23 footprint name change from Notecarrier-A.
Parts:
- Q2: footprint blues-kicad-lib:SOT23 -> blues-kicad-lib:SOT23_NO-FILL
Changed lines of the file:
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@@
       (effects (font (size 1.27 1.27)) (justify left))
     )
-    (property "Footprint" "blues-kicad-lib:SOT23" (at 140.97 236.855 0)
+    (property "Footprint" "blues-kicad-lib:SOT23_NO-FILL" (at 140.97 236.855 0)
       (effects (font (size 1.27 1.27) italic) (justify left) hide)
     )
@@
       (effects (font (size 1.27 1.27)) hide)
     )
+    (property "Critical" "" (at 146.05 234.95 0)
+      (effects (font (size 1.27 1.27)) hide)
+    )
+    (property "Manufacturer" "" (at 146.05 234.95 0)
+      (effects (font (size 1.27 1.27)) hide)
+    )
+    (property "Order Code" "" (at 146.05 234.95 0)
+      (effects (font (size 1.27 1.27)) hide)
+    )
+    (property "Part Number" "" (at 146.05 234.95 0)
+      (effects (font (size 1.27 1.27)) hide)
+    )
+    (property "Supplier" "" (at 146.05 234.95 0)
+      (effects (font (size 1.27 1.27)) hide)
+    )
