File: Notecarrier-A/KiCad_format/Notecarrier-A.kicad_sch (KiCad schematic)
At the start: 10 parts

Commit message: Release RevA of Notecarrier-A port.
Validation complete. Results in the validation directory, documented in PortingNotes.md.
Parts:
- FID1, FID2, FID3, FID4: footprint blues-kicad-lib:FIDUCIAL -> blues-kicad-lib:FIDUCIAL_MIN-CLEARANCE
Changed lines of the file:
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@@
   (title_block
     (title "Notecarrier-A")
-    (date "DRAFT")
+    (date "2023-05-23")
     (rev "A")
     (comment 1 "Blues Inc")
@@
       (effects (font (size 1.27 1.27)) (justify left) hide)
     )
-    (property "Footprint" "blues-kicad-lib:FIDUCIAL" (at 218.44 213.36 0)
+    (property "Footprint" "blues-kicad-lib:FIDUCIAL_MIN-CLEARANCE" (at 218.44 213.36 0)
       (effects (font (size 1.27 1.27)) hide)
     )
@@
     )
     (property "Distributor" "FAE" (at 218.44 213.36 0)
+      (effects (font (size 1.27 1.27)) hide)
+    )
+    (property "Critical" "" (at 218.44 213.36 0)
+      (effects (font (size 1.27 1.27)) hide)
+    )
+    (property "Manufacturer" "" (at 218.44 213.36 0)
+      (effects (font (size 1.27 1.27)) hide)
+    )
+    (property "Order Code" "" (at 218.44 213.36 0)
+      (effects (font (size 1.27 1.27)) hide)
+    )
+    (property "Part Number" "" (at 218.44 213.36 0)
+      (effects (font (size 1.27 1.27)) hide)
+    )
+    (property "Supplier" "" (at 218.44 213.36 0)
       (effects (font (size 1.27 1.27)) hide)
     )
@@
       (effects (font (size 1.27 1.27)) (justify left) hide)
     )
-    (property "Footprint" "blues-kicad-lib:FIDUCIAL" (at 212.09 213.36 0)
+    (property "Footprint" "blues-kicad-lib:FIDUCIAL_MIN-CLEARANCE" (at 212.09 213.36 0)
       (effects (font (size 1.27 1.27)) hide)
     )
@@
     )
     (property "Distributor" "FAE" (at 212.09 213.36 0)
+      (effects (font (size 1.27 1.27)) hide)
+    )
+    (property "Critical" "" (at 212.09 213.36 0)
+      (effects (font (size 1.27 1.27)) hide)
+    )
+    (property "Manufacturer" "" (at 212.09 213.36 0)
+      (effects (font (size 1.27 1.27)) hide)
+    )
+    (property "Order Code" "" (at 212.09 213.36 0)
+      (effects (font (size 1.27 1.27)) hide)
+    )
+    (property "Part Number" "" (at 212.09 213.36 0)
+      (effects (font (size 1.27 1.27)) hide)
+    )
+    (property "Supplier" "" (at 212.09 213.36 0)
       (effects (font (size 1.27 1.27)) hide)
     )
@@
       (effects (font (size 1.27 1.27)) (justify left) hide)
     )
-    (property "Footprint" "blues-kicad-lib:FIDUCIAL" (at 218.44 207.01 0)
+    (property "Footprint" "blues-kicad-lib:FIDUCIAL_MIN-CLEARANCE" (at 218.44 207.01 0)
       (effects (font (size 1.27 1.27)) hide)
     )
@@
     )
     (property "Distributor" "FAE" (at 218.44 207.01 0)
+      (effects (font (size 1.27 1.27)) hide)
+    )
+    (property "Critical" "" (at 218.44 207.01 0)
+      (effects (font (size 1.27 1.27)) hide)
+    )
+    (property "Manufacturer" "" (at 218.44 207.01 0)
+      (effects (font (size 1.27 1.27)) hide)
+    )
+    (property "Order Code" "" (at 218.44 207.01 0)
+      (effects (font (size 1.27 1.27)) hide)
+    )
+    (property "Part Number" "" (at 218.44 207.01 0)
+      (effects (font (size 1.27 1.27)) hide)
+    )
+    (property "Supplier" "" (at 218.44 207.01 0)
       (effects (font (size 1.27 1.27)) hide)
     )
@@
       (effects (font (size 1.27 1.27)) (justify left) hide)
     )
-    (property "Footprint" "blues-kicad-lib:FIDUCIAL" (at 212.09 207.01 0)
+    (property "Footprint" "blues-kicad-lib:FIDUCIAL_MIN-CLEARANCE" (at 212.09 207.01 0)
       (effects (font (size 1.27 1.27)) hide)
     )
@@
       (effects (font (size 1.27 1.27)) hide)
     )
+    (property "Critical" "" (at 212.09 207.01 0)
+      (effects (font (size 1.27 1.27)) hide)
+    )
+    (property "Manufacturer" "" (at 212.09 207.01 0)
+      (effects (font (size 1.27 1.27)) hide)
+    )
+    (property "Order Code" "" (at 212.09 207.01 0)
+      (effects (font (size 1.27 1.27)) hide)
+    )
+    (property "Part Number" "" (at 212.09 207.01 0)
+      (effects (font (size 1.27 1.27)) hide)
+    )
+    (property "Supplier" "" (at 212.09 207.01 0)
+      (effects (font (size 1.27 1.27)) hide)
+    )
