File: Notecarrier-A/v2.0/KiCad_format/Notecarrier-A_Power.kicad_sch (KiCad schematic)
At the start: 44 parts, among them J10 00711, J12 B2B-PH-SM4-TBT(LF)(SN), J19 10118192-0002LF, J19 NU, J3 B2B-PH-SM4-TBT(LF)(SN), J4 B2B-PH-SM4-TBT(LF)(SN), J9 12734, SW1 CJS-1200TA, U2 BQ24210DQCT, U3 MAX17225ELT, U4 TPS62748YFPT

Commit message: Upgrade the four original ports to KiCad 9; fix F v1.3 DRC; document F errata
Notecarrier-A v2.0, -B v2.1, -F v1.3 and -Pi v1.1 were authored in KiCad 7 and
are now upgraded in place (board 20221018 -> 20241229, schematics -> 20250114).
The upgrade is verified lossless on all four:

- every fabrication layer (copper, mask, paste, silk, Edge.Cuts) is
  geometrically identical before and after at 600 dpi, and drill files are
  textually identical;
- schematic netlists are unchanged - same components, same net partitions
  (A 99/114, B 62/87, F 110/166, Pi 46/95);
- kicanvas renders and the RAG extract both still pass.

Zones are NOT refilled - these ports depend on preserved fills.

Notecarrier-F: the board's 54 net-less 0.6 mm copper patches (footprint
weird-no-fill-via_Fv1.2) sit inside GND copper and are now assigned the GND net
they belong to. DRC goes from 171 errors to 0 with no change to any copper
geometry.

Notecarrier-F ERRATA.md (new): the power section does not match the shipped
board. U9 (AP2139AK-3.3 LDO) with C33/C34, and DS7 (STPS3H100U), are missing
from both schematic and board though they are in the Altium source, the released
BOM, the released pick-and-place, and the shipped copper/mask/paste. All six
diodes carry the wrong part and package: the released design uses FSV1045V in
TO277-3 (3 pads) for DS1/DS2/DS4/DS5 and STPS3H100U in SMB for DS3/DS6/DS7,
where the port has B360A-13-F in DO-214AC SMA (2 pads) throughout. The errata
records the exact wiring and coordinates needed to fix it. Flagged in the root
README and the port's README.

Also documented per port: the DRC exclusions recorded by KiCad 7 no longer
suppress anything, because KiCad 9 computes different marker keys. They are left
as the author's record and the remaining violations are explained in each
Porting-Notes - including evidence that A's J9 pad-vs-zone reports are
preserved-fill artifacts (its In1 plane matches the shipped GND film to within
0.9% of lit area), and that B's 4 error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
Parts:
- renumbered C13 to C1, C111 to C10, C112 to C11, C1 to C12, C2 to C13, C14 to C2, C15 to C3, C16 to C4, C116 to C5, C7 to C6, C8 to C7, C9 to C8, C10 to C9, DS14 to DS4, DS3 to DS5, DS4 to DS6, J19 to J11, J19 to J2, L4 to L1, R10 to R1, R4 to R10, R6 to R4, R307 to R5, R1 to R6, R2 to R8, R3 to R9, U4 to U1, U3 to U2, U2 to U3
