File: Notecarrier-Pi/v1.1/KiCad_format/Notecarrier-Pi.kicad_sch (KiCad schematic)
At the start: 47 parts, among them J1 2223, J3 MDT420E01001, J4 10118192-0002LF, J5 GROVE, J5 NanoSIM - SF72S006VBAR2500

Commit message: Upgrade the four original ports to KiCad 9; fix F v1.3 DRC; document F errata
Notecarrier-A v2.0, -B v2.1, -F v1.3 and -Pi v1.1 were authored in KiCad 7 and
are now upgraded in place (board 20221018 -> 20241229, schematics -> 20250114).
The upgrade is verified lossless on all four:

- every fabrication layer (copper, mask, paste, silk, Edge.Cuts) is
  geometrically identical before and after at 600 dpi, and drill files are
  textually identical;
- schematic netlists are unchanged - same components, same net partitions
  (A 99/114, B 62/87, F 110/166, Pi 46/95);
- kicanvas renders and the RAG extract both still pass.

Zones are NOT refilled - these ports depend on preserved fills.

Notecarrier-F: the board's 54 net-less 0.6 mm copper patches (footprint
weird-no-fill-via_Fv1.2) sit inside GND copper and are now assigned the GND net
they belong to. DRC goes from 171 errors to 0 with no change to any copper
geometry.

Notecarrier-F ERRATA.md (new): the power section does not match the shipped
board. U9 (AP2139AK-3.3 LDO) with C33/C34, and DS7 (STPS3H100U), are missing
from both schematic and board though they are in the Altium source, the released
BOM, the released pick-and-place, and the shipped copper/mask/paste. All six
diodes carry the wrong part and package: the released design uses FSV1045V in
TO277-3 (3 pads) for DS1/DS2/DS4/DS5 and STPS3H100U in SMB for DS3/DS6/DS7,
where the port has B360A-13-F in DO-214AC SMA (2 pads) throughout. The errata
records the exact wiring and coordinates needed to fix it. Flagged in the root
README and the port's README.

Also documented per port: the DRC exclusions recorded by KiCad 7 no longer
suppress anything, because KiCad 9 computes different marker keys. They are left
as the author's record and the remaining violations are explained in each
Porting-Notes - including evidence that A's J9 pad-vs-zone reports are
preserved-fill artifacts (its In1 plane matches the shipped GND film to within
0.9% of lit area), and that B's 4 error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
Parts:
- renumbered C3 to C4, C3 to C5, C3 to C6, J5 to J2, R5 to R1, R5 to R2, R5 to R3, R16 to R4, TVS2 to TVS4
