File: Mojo/v1.1/KiCad_format/Mojo.kicad_sch (KiCad schematic)
At the start: 22 parts, among them IC1 LTC2959IDDB#TRMPBF, J1 20404, J2 Header 2-Pin, 0.100 in, J3 Header 2-Pin, 0.100 in, J4 20404, J5 QWIIC SM04B-SRSS-TB(LF)(SN), J6 QWIIC SM04B-SRSS-TB(LF)(SN), J7 Header 2-Pin, 0.100 in, J8 Header 3-Pin, 0.100 in

Commit message: Ports: fill in the MPNs the old BOM gate was hiding
With the BOM comparator no longer treating a blank KiCad MPN as agreement, four
boards turned out to be missing manufacturer part numbers that their shipped
BOMs specify. None of this was visible before, because the comparison skipped
any refdes whose KiCad MPN was empty and then reported "BOM matches exactly".

  Cygnet          74 parts, none of which carried an MPN field at all
  Scoop           C3, U2, U4
  Notecarrier-XI  J9
  Mojo            R2, R3 - the only two parts on the board lacking the
                  MANUFACTURER PART NUMBER field their peers all carry

Filled from each board's own shipped BOM, which is authoritative for what was
built, using the field name that board's config already declares. There was no
conflict to resolve: the KiCad side held nothing.

Verified: all eight boards with a BOM gate now pass, every edited schematic
exports an identical netlist before and after, and kicanvas renders all of them.
Mojo's full battery is green end to end (ERC, DRC, BOM, gerber diff, placement,
kicanvas, RAG), with NETLIST skipped under its declared justification.

Co-Authored-By: Claude Fable 5 <noreply@anthropic.com>
Parts:
- R2, R3: MANUFACTURER PART NUMBER (none) -> RC0603FR-0722KL
Changed lines of the file:
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@@
 				(justify right bottom)
+			)
+		)		(property "MANUFACTURER PART NUMBER" "RC0603FR-0722KL"
+			(at 96.52 180.34 0)
+			(effects
+				(font
+					(size 1.27 1.27)
+				)
+				(hide yes)
 			)
 		)
@@
 				(justify right bottom)
 			)
-		)
+		)		(property "MANUFACTURER PART NUMBER" "RC0603FR-0722KL"
+			(at 127 180.34 0)
+			(effects
+				(font
+					(size 1.27 1.27)
+				)
+				(hide yes)
+			)
+		)
