File: Cygnet/v1.2/KiCad_format/Cygnet_Feather-Connector.kicad_sch (KiCad schematic)
At the start: 8 parts, among them J1 12402012E212A

Commit message: Ports: fill in the MPNs the old BOM gate was hiding
With the BOM comparator no longer treating a blank KiCad MPN as agreement, four
boards turned out to be missing manufacturer part numbers that their shipped
BOMs specify. None of this was visible before, because the comparison skipped
any refdes whose KiCad MPN was empty and then reported "BOM matches exactly".

  Cygnet          74 parts, none of which carried an MPN field at all
  Scoop           C3, U2, U4
  Notecarrier-XI  J9
  Mojo            R2, R3 - the only two parts on the board lacking the
                  MANUFACTURER PART NUMBER field their peers all carry

Filled from each board's own shipped BOM, which is authoritative for what was
built, using the field name that board's config already declares. There was no
conflict to resolve: the KiCad side held nothing.

Verified: all eight boards with a BOM gate now pass, every edited schematic
exports an identical netlist before and after, and kicanvas renders all of them.
Mojo's full battery is green end to end (ERC, DRC, BOM, gerber diff, placement,
kicanvas, RAG), with NETLIST skipped under its declared justification.

Co-Authored-By: Claude Fable 5 <noreply@anthropic.com>
Parts:
- C32: MPN (none) -> cs1206kkx7rcbb103
- C33: MPN (none) -> cc0402krx7r7bb104
- J1: MPN (none) -> 12402012e212a
- R20, R21: MPN (none) -> rc0402jr-075k1l
- R22: MPN (none) -> rc1206fr-071ml
Changed lines of the file:
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@@
 				(justify left bottom)
+			)
+		)		(property "MPN" "cc0402krx7r7bb104"
+			(at 177 242.0662 0)
+			(effects
+				(font
+					(size 1.27 1.27)
+				)
+				(hide yes)
 			)
 		)
@@
 				(justify right bottom)
 			)
+		)		(property "MPN" "12402012e212a"
+			(at 317.579 57.0022 0)
+			(effects
+				(font
+					(size 1.27 1.27)
+				)
+				(hide yes)
+			)
 		)
 		(property "Footprint" "Cygnet-altium-import:AMPHENOL_12402012E212A"
@@
 				(justify right bottom)
 			)
+		)		(property "MPN" "rc0402jr-075k1l"
+			(at 269.379 39.4632 0)
+			(effects
+				(font
+					(size 1.27 1.27)
+				)
+				(hide yes)
+			)
 		)
 		(property "Footprint" "Cygnet-altium-import:RESC1005X40X25NL05T10"
@@
 				(justify right bottom)
 			)
+		)		(property "MPN" "rc1206fr-071ml"
+			(at 356.499 80.0022 0)
+			(effects
+				(font
+					(size 1.27 1.27)
+				)
+				(hide yes)
+			)
 		)
 		(property "Footprint" "Cygnet-altium-import:RC1206FR-071ML-Footprint-1"
@@
 				(justify right bottom)
 			)
+		)		(property "MPN" "cs1206kkx7rcbb103"
+			(at 356.999 76.0022 0)
+			(effects
+				(font
+					(size 1.27 1.27)
+				)
+				(hide yes)
+			)
 		)
 		(property "Footprint" "Cygnet-altium-import:CS1206KKX7RCBB103-Footprint-1"
@@
 				(justify right bottom)
 			)
-		)
+		)		(property "MPN" "rc0402jr-075k1l"
+			(at 364.459 55.9622 0)
+			(effects
+				(font
+					(size 1.27 1.27)
+				)
+				(hide yes)
+			)
+		)

Commit message: Ports: restore shipped-BOM letter case in the backfilled MPN fields
The 78-MPN backfill (d1a1499) said "filled from each board's own shipped BOM"
but inserted the comparison's casefolded text, not the spreadsheets' - every
shipped BOM involved is uppercase (SKRPADE010, CC0603KRX7R7BB105,
TSW-105-07-F-D), and the gate only agreed because its comparison is
case-insensitive. The lowercase text was user-visible in the schematic fields
and flowed into the RAG extract's new MPN column.

Restored the spreadsheets' exact text on all 78 fields (Cygnet 74, Scoop 3,
XI 1; Mojo's two were inserted correctly), scoped to exactly the property
values that commit added. Verified inert: the BOM gate passes on all three
boards and the re-exported netlists differ only in the affected field text.

Co-Authored-By: Claude Fable 5 <noreply@anthropic.com>
Parts:
- C32: MPN cs1206kkx7rcbb103 -> CS1206KKX7RCBB103
- C33: MPN cc0402krx7r7bb104 -> CC0402KRX7R7BB104
- J1: MPN 12402012e212a -> 12402012E212A
- R20, R21: MPN rc0402jr-075k1l -> RC0402JR-075K1L
- R22: MPN rc1206fr-071ml -> RC1206FR-071ML
Changed lines of the file:
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@@
 				(justify left bottom)
 			)
-		)		(property "MPN" "cc0402krx7r7bb104"
+		)		(property "MPN" "CC0402KRX7R7BB104"
 			(at 177 242.0662 0)
 			(effects
@@
 				(justify right bottom)
 			)
-		)		(property "MPN" "12402012e212a"
+		)		(property "MPN" "12402012E212A"
 			(at 317.579 57.0022 0)
 			(effects
@@
 				(justify right bottom)
 			)
-		)		(property "MPN" "rc0402jr-075k1l"
+		)		(property "MPN" "RC0402JR-075K1L"
 			(at 269.379 39.4632 0)
 			(effects
@@
 				(justify right bottom)
 			)
-		)		(property "MPN" "rc1206fr-071ml"
+		)		(property "MPN" "RC1206FR-071ML"
 			(at 356.499 80.0022 0)
 			(effects
@@
 				(justify right bottom)
 			)
-		)		(property "MPN" "cs1206kkx7rcbb103"
+		)		(property "MPN" "CS1206KKX7RCBB103"
 			(at 356.999 76.0022 0)
 			(effects
@@
 				(justify right bottom)
 			)
-		)		(property "MPN" "rc0402jr-075k1l"
+		)		(property "MPN" "RC0402JR-075K1L"
 			(at 364.459 55.9622 0)
 			(effects
