File: Cygnet/v1.2/KiCad_format/Cygnet_Power.kicad_sch (KiCad schematic)
At the start: 34 parts, among them J6 1769 - JST-PH 2-PIN SMT, U2 TPS63020DSJT, U3 ISL9122AIINZ-T, U4 LM66200DRLR, U5 MCP73831-2ACI/MC, U6 AP2139AK-3.3TRG1

Commit message: Ports: fill in the MPNs the old BOM gate was hiding
With the BOM comparator no longer treating a blank KiCad MPN as agreement, four
boards turned out to be missing manufacturer part numbers that their shipped
BOMs specify. None of this was visible before, because the comparison skipped
any refdes whose KiCad MPN was empty and then reported "BOM matches exactly".

  Cygnet          74 parts, none of which carried an MPN field at all
  Scoop           C3, U2, U4
  Notecarrier-XI  J9
  Mojo            R2, R3 - the only two parts on the board lacking the
                  MANUFACTURER PART NUMBER field their peers all carry

Filled from each board's own shipped BOM, which is authoritative for what was
built, using the field name that board's config already declares. There was no
conflict to resolve: the KiCad side held nothing.

Verified: all eight boards with a BOM gate now pass, every edited schematic
exports an identical netlist before and after, and kicanvas renders all of them.
Mojo's full battery is green end to end (ERC, DRC, BOM, gerber diff, placement,
kicanvas, RAG), with NETLIST skipped under its declared justification.

Co-Authored-By: Claude Fable 5 <noreply@anthropic.com>
Parts:
- C17, C18, C22, C23: MPN (none) -> grm188r61a106ke69d
- C19, C20: MPN (none) -> f930j107kaabe1
- C21, C28, C30: MPN (none) -> grm033r61c104ke84j
- C24, C25, C29, C31: MPN (none) -> c0402b105k016t
- C26, C27: MPN (none) -> cl10a475kp8nnnc
- L1: MPN (none) -> mckk1608t1r0mn
- L2: MPN (none) -> xfl4020-152mec
- LD2: MPN (none) -> sml-p12wtt86r
- R11: MPN (none) -> rc0402fr-071kl
- R12, R15: MPN (none) -> rc0201fr-071ml
- R14: MPN (none) -> mc0201l6f1002se
- R16: MPN (none) -> mr02x1803fal
- R17: MPN (none) -> crcw02011k00fned
- R18: MPN (none) -> crcw02012k80fked
- R19: MPN (none) -> crcw02018m20fned
- TVS4: MPN (none) -> sm6t6v8a
- U2: MPN (none) -> tps63020dsjt
- U3: MPN (none) -> isl9122aiinz-t
- U4: MPN (none) -> lm66200drlr
- U5: MPN (none) -> mcp73831-2aci/mc

Commit message: Ports: restore shipped-BOM letter case in the backfilled MPN fields
The 78-MPN backfill (d1a1499) said "filled from each board's own shipped BOM"
but inserted the comparison's casefolded text, not the spreadsheets' - every
shipped BOM involved is uppercase (SKRPADE010, CC0603KRX7R7BB105,
TSW-105-07-F-D), and the gate only agreed because its comparison is
case-insensitive. The lowercase text was user-visible in the schematic fields
and flowed into the RAG extract's new MPN column.

Restored the spreadsheets' exact text on all 78 fields (Cygnet 74, Scoop 3,
XI 1; Mojo's two were inserted correctly), scoped to exactly the property
values that commit added. Verified inert: the BOM gate passes on all three
boards and the re-exported netlists differ only in the affected field text.

Co-Authored-By: Claude Fable 5 <noreply@anthropic.com>
Parts:
- C17, C18, C22, C23: MPN grm188r61a106ke69d -> GRM188R61A106KE69D
- C19, C20: MPN f930j107kaabe1 -> F930J107KAABE1
- C21, C28, C30: MPN grm033r61c104ke84j -> GRM033R61C104KE84J
- C24, C25, C29, C31: MPN c0402b105k016t -> C0402B105K016T
- C26, C27: MPN cl10a475kp8nnnc -> CL10A475KP8NNNC
- L1: MPN mckk1608t1r0mn -> MCKK1608T1R0MN
- L2: MPN xfl4020-152mec -> XFL4020-152MEC
- LD2: MPN sml-p12wtt86r -> SML-P12WTT86R
- R11: MPN rc0402fr-071kl -> RC0402FR-071KL
- R12, R15: MPN rc0201fr-071ml -> RC0201FR-071ML
- R14: MPN mc0201l6f1002se -> MC0201L6F1002SE
- R16: MPN mr02x1803fal -> MR02X1803FAL
- R17: MPN crcw02011k00fned -> CRCW02011K00FNED
- R18: MPN crcw02012k80fked -> CRCW02012K80FKED
- R19: MPN crcw02018m20fned -> CRCW02018M20FNED
- TVS4: MPN sm6t6v8a -> SM6T6V8A
- U2: MPN tps63020dsjt -> TPS63020DSJT
- U3: MPN isl9122aiinz-t -> ISL9122AIINZ-T
- U4: MPN lm66200drlr -> LM66200DRLR
- U5: MPN mcp73831-2aci/mc -> MCP73831-2ACI/MC
Changed lines of the file:
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@@
 				(justify left bottom)
 			)
-		)		(property "MPN" "grm033r61c104ke84j"
+		)		(property "MPN" "GRM033R61C104KE84J"
 			(at 55 262.0022 0)
 			(effects
@@
 				(justify left bottom)
 			)
-		)		(property "MPN" "cl10a475kp8nnnc"
+		)		(property "MPN" "CL10A475KP8NNNC"
 			(at 312.5 191.0662 0)
 			(effects
@@
 				(justify left bottom)
 			)
-		)		(property "MPN" "cl10a475kp8nnnc"
+		)		(property "MPN" "CL10A475KP8NNNC"
 			(at 320 191.0662 0)
 			(effects
@@
 				(justify left bottom)
 			)
-		)		(property "MPN" "sm6t6v8a"
+		)		(property "MPN" "SM6T6V8A"
 			(at 102.5 106.7622 0)
 			(effects
@@
 				(justify left bottom)
 			)
-		)		(property "MPN" "c0402b105k016t"
+		)		(property "MPN" "C0402B105K016T"
 			(at 102.5 262.0022 0)
 			(effects
@@
 				(justify right bottom)
 			)
-		)		(property "MPN" "crcw02011k00fned"
+		)		(property "MPN" "CRCW02011K00FNED"
 			(at 377.46 164.6222 0)
 			(effects
@@
 				(justify left bottom)
 			)
-		)		(property "MPN" "f930j107kaabe1"
+		)		(property "MPN" "F930J107KAABE1"
 			(at 307.34 86.1822 0)
 			(effects
@@
 				(justify left bottom)
 			)
-		)		(property "MPN" "c0402b105k016t"
+		)		(property "MPN" "C0402B105K016T"
 			(at 40 109.5022 0)
 			(effects
@@
 				(justify left bottom)
 			)
-		)		(property "MPN" "grm188r61a106ke69d"
+		)		(property "MPN" "GRM188R61A106KE69D"
 			(at 375 82.0022 0)
 			(effects
@@
 				(justify right bottom)
 			)
-		)		(property "MPN" "mcp73831-2aci/mc"
+		)		(property "MPN" "MCP73831-2ACI/MC"
 			(at 330 162.0022 0)
 			(effects
@@
 				(justify right bottom)
 			)
-		)		(property "MPN" "mckk1608t1r0mn"
+		)		(property "MPN" "MCKK1608T1R0MN"
 			(at 172.5 69.5022 0)
 			(effects
@@
 				(justify right bottom)
 			)
-		)		(property "MPN" "lm66200drlr"
+		)		(property "MPN" "LM66200DRLR"
 			(at 55 87.0022 0)
 			(effects
@@
 				(justify right bottom)
 			)
-		)		(property "MPN" "mc0201l6f1002se"
+		)		(property "MPN" "MC0201L6F1002SE"
 			(at 44.96 81.9622 0)
 			(effects
@@
 				(justify left bottom)
 			)
-		)		(property "MPN" "c0402b105k016t"
+		)		(property "MPN" "C0402B105K016T"
 			(at 30 109.5022 0)
 			(effects
@@
 				(justify left bottom)
 			)
-		)		(property "MPN" "c0402b105k016t"
+		)		(property "MPN" "C0402B105K016T"
 			(at 60.96 261.4022 0)
 			(effects
@@
 				(justify left bottom)
 			)
-		)		(property "MPN" "grm033r61c104ke84j"
+		)		(property "MPN" "GRM033R61C104KE84J"
 			(at 97.5 259.5022 0)
 			(effects
@@
 				(justify right bottom)
 			)
-		)		(property "MPN" "crcw02012k80fked"
+		)		(property "MPN" "CRCW02012K80FKED"
 			(at 362.46 184.6222 0)
 			(effects
@@
 				(justify left bottom)
 			)
-		)		(property "MPN" "grm033r61c104ke84j"
+		)		(property "MPN" "GRM033R61C104KE84J"
 			(at 322.58 83.6822 0)
 			(effects
@@
 				(justify right bottom)
 			)
-		)		(property "MPN" "tps63020dsjt"
+		)		(property "MPN" "TPS63020DSJT"
 			(at 342.74 34.5822 0)
 			(effects
@@
 				(justify right bottom)
 			)
-		)		(property "MPN" "rc0402fr-071kl"
+		)		(property "MPN" "RC0402FR-071KL"
 			(at 287.5 44.5022 0)
 			(effects
@@
 				(justify left bottom)
 			)
-		)		(property "MPN" "sml-p12wtt86r"
+		)		(property "MPN" "SML-P12WTT86R"
 			(at 345.52 149.6822 0)
 			(effects
@@
 				(justify left bottom)
 			)
-		)		(property "MPN" "grm188r61a106ke69d"
+		)		(property "MPN" "GRM188R61A106KE69D"
 			(at 147.5 101.0662 0)
 			(effects
@@
 				(justify right bottom)
 			)
-		)		(property "MPN" "mr02x1803fal"
+		)		(property "MPN" "MR02X1803FAL"
 			(at 317.5 83.5622 0)
 			(effects
@@
 				(justify right bottom)
 			)
-		)		(property "MPN" "isl9122aiinz-t"
+		)		(property "MPN" "ISL9122AIINZ-T"
 			(at 175.16 82.0022 0)
 			(effects
@@
 				(justify right bottom)
 			)
-		)		(property "MPN" "xfl4020-152mec"
+		)		(property "MPN" "XFL4020-152MEC"
 			(at 340 69.5022 0)
 			(effects
@@
 				(justify right bottom)
 			)
-		)		(property "MPN" "rc0201fr-071ml"
+		)		(property "MPN" "RC0201FR-071ML"
 			(at 384.96 82.1222 0)
 			(effects
@@
 				(justify right bottom)
 			)
-		)		(property "MPN" "crcw02018m20fned"
+		)		(property "MPN" "CRCW02018M20FNED"
 			(at 45 244.5022 0)
 			(effects
@@
 				(justify left bottom)
 			)
-		)		(property "MPN" "f930j107kaabe1"
+		)		(property "MPN" "F930J107KAABE1"
 			(at 302.26 86.1822 0)
 			(effects
@@
 				(justify right bottom)
 			)
-		)		(property "MPN" "rc0201fr-071ml"
+		)		(property "MPN" "RC0201FR-071ML"
 			(at 314.96 55.7022 0)
 			(effects
@@
 				(justify left bottom)
 			)
-		)		(property "MPN" "grm188r61a106ke69d"
+		)		(property "MPN" "GRM188R61A106KE69D"
 			(at 370 82.0022 0)
 			(effects
@@
 				(justify left bottom)
 			)
-		)		(property "MPN" "grm188r61a106ke69d"
+		)		(property "MPN" "GRM188R61A106KE69D"
 			(at 202.5 101.0662 0)
 			(effects

Commit message: Ports: convert design-note text_boxes to plain text so kicanvas can render them
kicanvas parses text_box but never paints it - true of the current upstream
build too, which is byte-identical to the one vendored here. On the published
datasheet pages that left the design notes (charger limits, regulator specs,
population notes) as empty frames, and on Cygnet, whose note frames ARE the
text_boxes, the notes were entirely invisible. KiCad renders plain text and
rectangles identically to what it drew before, and kicanvas renders both, so
the 28 text_boxes across 12 sheets on 6 boards become plain text items - plus a
synthesized rectangle carrying the exact stroke and fill for the 5 Cygnet notes
whose box itself is visible (yellow-filled with a border).

Two things made this more than a mechanical swap:

- text_box soft-wraps and plain text does not. A first attempt left two notes
  overflowing their frames and colliding with a neighbouring note. The wrap is
  now frozen at exactly the line breaks KiCad itself used: each sheet's
  before-conversion PDF carries a hidden searchable text layer, and the
  converter reads the wrapped lines out of the note's own rectangle, guarded by
  a word-for-word equality check against the source text. That guard earned its
  keep twice, catching part-number labels that physically overlap two of the
  note boxes.

- kicanvas draws default-colored text in its theme color, which is white - and
  two Cygnet notes sit on yellow fills. Those five framed notes now carry an
  explicit (0,0,193) font color, sampled from KiCad's own plot of the same
  notes, so KiCad's output is unchanged and kicanvas is readable.

Verified per board: netlists byte-equal before and after; KiCad PDF renders
differ only by sub-millimetre line pitch (0.05-0.7% of sampled pixels, every
note inside its frame - checked visually on the worst sheets); kicanvas renders
all 12 sheets with the notes now visible; committed screenshots regenerated,
all six boards PASS.

Co-Aut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
Other:
- note added: "CURRENT LEGEND 2A: +VMAIN, GND 1A: +VIN, +VBAT 500mA: +3V3_OUT, +VUSB, +VIO 250mA: +3V3_VUSB, +3V3_CONN < 20 mA: GPIO/ control pins"
- note added: "Iqmax=1.5uA Isdmax=1uA VEN-IH=1.2V VEN-IL=0.3V IPD-EN=0.2uA"
- note added: "LIPO BATTERY 3.3V - 4.2V"
- note added: "Note: Do not mount/ populate R14"
Changed lines of the file:
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@@
 		)
 	)
-	(text_box "Iqmax=1.5uA\nIsdmax=1uA\nVEN-IH=1.2V\nVEN-IL=0.3V\nIPD-EN=0.2uA"
+	(text "Iqmax=1.5uA\nIsdmax=1uA\nVEN-IH=1.2V\nVEN-IL=0.3V\nIPD-EN=0.2uA"
 		(exclude_from_sim no)
-		(at 89.408 250.0122 0)
-		(size -18.288 13.97)
-		(margins 0.9525 0.9525 0.9525 0.9525)
-		(stroke
-			(width -0.0001)
-			(type default)
-			(color 0 0 0 1)
-		)
-		(fill
-			(type none)
-		)
+		(at 72.0725 250.965 0)
 		(effects
 			(font
@@
 		)
 	)
-	(text_box "LIPO BATTERY\n3.3V - 4.2V"
+	(text "LIPO BATTERY\n3.3V - 4.2V"
 		(exclude_from_sim no)
-		(at 302.768 156.7942 0)
-		(size -18.288 5.588)
-		(margins 0.9525 0.9525 0.9525 0.9525)
-		(stroke
-			(width -0.0001)
-			(type default)
-			(color 0 0 0 1)
-		)
-		(fill
-			(type none)
-		)
+		(at 285.432 157.747 0)
 		(effects
 			(font
@@
 		)
 	)
-	(text_box "Note: Do not mount/ populate R14"
-		(exclude_from_sim no)
-		(at 75 72.0022 0)
-		(size -22.5 7.5)
-		(margins 0.9525 0.9525 0.9525 0.9525)
+	(rectangle
+		(start 52.5 72.0022)
+		(end 75 79.5022)
 		(stroke
 			(width 0)
@@
 			(color 255 255 150 1)
 		)
+	)
+	(text "Note: Do not\nmount/ populate\nR14"
+		(exclude_from_sim no)
+		(at 53.4525 72.9547 0)
 		(effects
 			(font
 				(size 1.27 1.27)
+				(color 0 0 193 1)
 			)
 			(justify left top)
 		)
 	)
-	(text_box "CURRENT LEGEND\n2A: +VMAIN, GND\n1A: +VIN, +VBAT\n500mA: +3V3_OUT, +VUSB, +VIO \n250mA: +3V3_VUSB, +3V3_CONN\n\n < 20 mA: GPIO/ control pins"
-		(exclude_from_sim no)
-		(at 242.4 142.5422 0)
-		(size -90 30)
-		(margins 0.9525 0.9525 0.9525 0.9525)
+	(rectangle
+		(start 152.4 142.542)
+		(end 242.4 172.542)
 		(stroke
 			(width 0)
@@
 			(color 255 255 150 1)
 		)
+	)
+	(text "CURRENT LEGEND\n2A: +VMAIN, GND\n1A: +VIN, +VBAT\n500mA: +3V3_OUT, +VUSB, +VIO\n250mA: +3V3_VUSB, +3V3_CONN\n\n< 20 mA: GPIO/ control pins"
+		(exclude_from_sim no)
+		(at 153.352 143.495 0)
 		(effects
 			(font
 				(size 1.778 1.778)
+				(color 0 0 193 1)
 			)
 			(justify left top)
