File: Cygnet/v1.2/KiCad_format/Cygnet_CPU.kicad_sch (KiCad schematic)
At the start: 38 parts, among them J4 BM04B-SRSS-TBT(LF)(SN), J5 FTSH-107-01-L-DV-K, SW1 PB-SKRPADE010, SW2 PB-SKRPABE010, SW3 PB-SKRPADE010, U1 STM32L433, Y1 ABS06-107-32.768KHZ-T

Commit message: fixes based on incorrect bom for cygnet mcu
Parts:
- U1: MPN STM32L433CB -> STM32L433CCT6
Changed lines of the file:
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@@
 				(justify right bottom)
 			)
-		)		(property "MPN" "STM32L433CB"
+		)		(property "MPN" "STM32L433CCT6"
 			(at 220 62.0022 0)
 			(effects
@@
 			)
 		)
-		(property "Description" "Ultra-low-power with FPU ARM Cortex-M4 MCU 80 MHz with 128 Kbytes Flash, USB FS, LCD"
+		(property "Description" "Ultra-low-power with FPU ARM Cortex-M4 MCU 80 MHz with 256 Kbytes Flash, USB FS, LCD"
 			(at 220 62.0022 0)
 			(effects
