File: Notecarrier-XI/v1.4/KiCad_format/Notecarrier-XI_Starnote-Connection.kicad_sch (KiCad schematic)
At the start: 19 parts, among them J6 MDT420E01001, J9 STRIP 5Px2 - MDT, P5 12402012E212A, SW1 EVP-BB2A9B000, SW2 EVP-BB2A9B000

Commit message: Ports: fill in the MPNs the old BOM gate was hiding
With the BOM comparator no longer treating a blank KiCad MPN as agreement, four
boards turned out to be missing manufacturer part numbers that their shipped
BOMs specify. None of this was visible before, because the comparison skipped
any refdes whose KiCad MPN was empty and then reported "BOM matches exactly".

  Cygnet          74 parts, none of which carried an MPN field at all
  Scoop           C3, U2, U4
  Notecarrier-XI  J9
  Mojo            R2, R3 - the only two parts on the board lacking the
                  MANUFACTURER PART NUMBER field their peers all carry

Filled from each board's own shipped BOM, which is authoritative for what was
built, using the field name that board's config already declares. There was no
conflict to resolve: the KiCad side held nothing.

Verified: all eight boards with a BOM gate now pass, every edited schematic
exports an identical netlist before and after, and kicanvas renders all of them.
Mojo's full battery is green end to end (ERC, DRC, BOM, gerber diff, placement,
kicanvas, RAG), with NETLIST skipped under its declared justification.

Co-Authored-By: Claude Fable 5 <noreply@anthropic.com>
Parts:
- J9: MANUFACTURER PART NUMBER (none) -> tsw-105-07-f-d
Changed lines of the file:
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@@
 				(justify right top)
+			)
+		)		(property "MANUFACTURER PART NUMBER" "tsw-105-07-f-d"
+			(at 120.65 210.6422 0)
+			(effects
+				(font
+					(size 1.27 1.27)
+				)
+				(hide yes)
 			)
 		)

Commit message: Ports: restore shipped-BOM letter case in the backfilled MPN fields
The 78-MPN backfill (d1a1499) said "filled from each board's own shipped BOM"
but inserted the comparison's casefolded text, not the spreadsheets' - every
shipped BOM involved is uppercase (SKRPADE010, CC0603KRX7R7BB105,
TSW-105-07-F-D), and the gate only agreed because its comparison is
case-insensitive. The lowercase text was user-visible in the schematic fields
and flowed into the RAG extract's new MPN column.

Restored the spreadsheets' exact text on all 78 fields (Cygnet 74, Scoop 3,
XI 1; Mojo's two were inserted correctly), scoped to exactly the property
values that commit added. Verified inert: the BOM gate passes on all three
boards and the re-exported netlists differ only in the affected field text.

Co-Authored-By: Claude Fable 5 <noreply@anthropic.com>
Parts:
- J9: MANUFACTURER PART NUMBER tsw-105-07-f-d -> TSW-105-07-F-D
Changed lines of the file:
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@@
 				(justify right top)
 			)
-		)		(property "MANUFACTURER PART NUMBER" "tsw-105-07-f-d"
+		)		(property "MANUFACTURER PART NUMBER" "TSW-105-07-F-D"
 			(at 120.65 210.6422 0)
 			(effects
