File: Notecarrier-XI/v1.4/KiCad_format/Notecarrier-XI_Power.kicad_sch (KiCad schematic)
At the start: 42 parts, among them U1 ISL9122AIRNZ-T, U2 LTC3128EUFD#PBF, U3 BQ25628ERYKR

Commit message: Ports: convert design-note text_boxes to plain text so kicanvas can render them
kicanvas parses text_box but never paints it - true of the current upstream
build too, which is byte-identical to the one vendored here. On the published
datasheet pages that left the design notes (charger limits, regulator specs,
population notes) as empty frames, and on Cygnet, whose note frames ARE the
text_boxes, the notes were entirely invisible. KiCad renders plain text and
rectangles identically to what it drew before, and kicanvas renders both, so
the 28 text_boxes across 12 sheets on 6 boards become plain text items - plus a
synthesized rectangle carrying the exact stroke and fill for the 5 Cygnet notes
whose box itself is visible (yellow-filled with a border).

Two things made this more than a mechanical swap:

- text_box soft-wraps and plain text does not. A first attempt left two notes
  overflowing their frames and colliding with a neighbouring note. The wrap is
  now frozen at exactly the line breaks KiCad itself used: each sheet's
  before-conversion PDF carries a hidden searchable text layer, and the
  converter reads the wrapped lines out of the note's own rectangle, guarded by
  a word-for-word equality check against the source text. That guard earned its
  keep twice, catching part-number labels that physically overlap two of the
  note boxes.

- kicanvas draws default-colored text in its theme color, which is white - and
  two Cygnet notes sit on yellow fills. Those five framed notes now carry an
  explicit (0,0,193) font color, sampled from KiCad's own plot of the same
  notes, so KiCad's output is unchanged and kicanvas is readable.

Verified per board: netlists byte-equal before and after; KiCad PDF renders
differ only by sub-millimetre line pitch (0.05-0.7% of sampled pixels, every
note inside its frame - checked visually on the worst sheets); kicanvas renders
all 12 sheets with the notes now visible; committed screenshots regenerated,
all six boards PASS.

Co-Aut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
Other:
- note added: "DESIGN NOTE: Charger: - Default charging voltage: 4.2V - Default charging current: 320mA - Default termination current: 20mA - Default pre-charge current: 20mA - No battery thermal protection"
- note added: "DESIGN NOTE: Input Voltage: 1.8V - 5.5V Output Voltage: 3.3V Peak Output Current: 500mA Average Current: 100mA"
- note added: "DESIGN NOTE: Power Path: - Input current limit: 3.5A - 26mOhm reverse blocking transistor - 15mOhm battery transistor Buck Regulator: - 1.5MHz frequency - Input Voltage: 5V - Output Voltage: 3.3-4.2V - Peak current: 2.5A"
Changed lines of the file:
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@@
 		)
 	)
-	(text_box "DESIGN NOTE:\nInput Voltage: 1.8V - 5.5V\nOutput Voltage: 3.3V\n\nPeak Output Current: 500mA\nAverage Current: 100mA"
+	(text "DESIGN NOTE:\nInput Voltage: 1.8V - 5.5V\nOutput Voltage: 3.3V\n\nPeak Output Current:\n500mA\nAverage Current: 100mA"
 		(exclude_from_sim no)
-		(at 224.995 57.5932 0)
-		(size -24.13 12.7)
-		(margins 0.9525 0.9525 0.9525 0.9525)
-		(stroke
-			(width -0.0001)
-			(type default)
-			(color 0 0 0 1)
-		)
-		(fill
-			(type none)
-		)
+		(at 201.817 58.5457 0)
 		(effects
 			(font
@@
 		)
 	)
-	(text_box "DESIGN NOTE:\n\nCharger:\n- Default charging voltage: 4.2V\n- Default charging current: 320mA\n- Default termination current: 20mA\n- Default pre-charge current: 20mA\n- No battery thermal protection"
+	(text "DESIGN NOTE:\n\nCharger:\n- Default charging voltage: 4.2V\n- Default charging current: 320mA\n- Default termination current: 20mA\n- Default pre-charge current: 20mA\n- No battery thermal protection"
 		(exclude_from_sim no)
-		(at 64.77 130.6322 0)
-		(size -33.02 16.51)
-		(margins 0.9525 0.9525 0.9525 0.9525)
-		(stroke
-			(width -0.0001)
-			(type default)
-			(color 0 0 0 1)
-		)
-		(fill
-			(type none)
-		)
+		(at 32.7025 131.585 0)
 		(effects
 			(font
@@
 		)
 	)
-	(text_box "DESIGN NOTE:\n\nPower Path:\n- Input current limit: 3.5A\n- 26mOhm reverse blocking transistor\n- 15mOhm battery transistor\n\nBuck Regulator:\n- 1.5MHz frequency\n- Input Voltage: 5V\n- Output Voltage: 3.3-4.2V\n- Peak current: 2.5A"
+	(text "DESIGN NOTE:\n\nPower Path:\n- Input current limit: 3.5A\n- 26mOhm reverse blocking transistor\n- 15mOhm battery transistor\n\nBuck Regulator:\n- 1.5MHz frequency\n- Input Voltage: 5V\n- Output Voltage: 3.3-4.2V\n- Peak current: 2.5A"
 		(exclude_from_sim no)
-		(at 124.46 121.7422 0)
-		(size -33.02 26.67)
-		(margins 0.9525 0.9525 0.9525 0.9525)
-		(stroke
-			(width -0.0001)
-			(type default)
-			(color 0 0 0 1)
-		)
-		(fill
-			(type none)
-		)
+		(at 92.3925 122.695 0)
 		(effects
 			(font
