File: Scoop/v1.0/KiCad_format/Scoop.kicad_sch (KiCad schematic)
At the start: 29 parts, among them J1 S2B-PH-SM4-TB(LF)(SN), J2 S2B-PH-SM4-TB(LF)(SN), J3 Header 2-Pin, 0.100 inch (0.2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, J4 Header 2-Pin, 0.100 inch (0.2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, J5 Header 2-Pin, 0.100 inch (0.2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, J6 Header 2-Pin, 0.100 inch (0.2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, U1 NCP718BSNADJT1G, U2 MAX40203AUK+T, U3 BD49K25G-TL, U4 MAX40203AUK+T

Commit message: Ports: restore shipped-BOM letter case in the backfilled MPN fields
The 78-MPN backfill (d1a1499) said "filled from each board's own shipped BOM"
but inserted the comparison's casefolded text, not the spreadsheets' - every
shipped BOM involved is uppercase (SKRPADE010, CC0603KRX7R7BB105,
TSW-105-07-F-D), and the gate only agreed because its comparison is
case-insensitive. The lowercase text was user-visible in the schematic fields
and flowed into the RAG extract's new MPN column.

Restored the spreadsheets' exact text on all 78 fields (Cygnet 74, Scoop 3,
XI 1; Mojo's two were inserted correctly), scoped to exactly the property
values that commit added. Verified inert: the BOM gate passes on all three
boards and the re-exported netlists differ only in the affected field text.

Co-Authored-By: Claude Fable 5 <noreply@anthropic.com>
Parts:
- C3: MANUFACTURER PART NUMBER cc0603krx7r7bb105 -> CC0603KRX7R7BB105
- U2, U4: MANUFACTURER PART NUMBER max40203auk+t -> MAX40203AUK+T
Changed lines of the file:
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@@
 				(justify right bottom)
 			)
-		)		(property "MANUFACTURER PART NUMBER" "max40203auk+t"
+		)		(property "MANUFACTURER PART NUMBER" "MAX40203AUK+T"
 			(at 261.62 101.6 0)
 			(effects
@@
 				(hide yes)
 			)
-		)		(property "MANUFACTURER PART NUMBER" "cc0603krx7r7bb105"
+		)		(property "MANUFACTURER PART NUMBER" "CC0603KRX7R7BB105"
 			(at 187.96 109.22 0)
 			(effects
@@
 				(justify right bottom)
 			)
-		)		(property "MANUFACTURER PART NUMBER" "max40203auk+t"
+		)		(property "MANUFACTURER PART NUMBER" "MAX40203AUK+T"
 			(at 142.24 101.6 0)
 			(effects
