File: Notecarrier-A/v2.3/KiCad_format/Notecarrier-A_Power.kicad_sch (KiCad schematic)
At the start: 45 parts, among them J10 00711, J11 12402012E212A, J12 B2B-PH-SM4-TBT(LF)(SN), J3 B2B-PH-SM4-TBT(LF)(SN), J4 B2B-PH-SM4-TBT(LF)(SN), J9 12734, SW1 CJS-1200TA, U1 TPS62748YFPT, U2 MAX17225ELT, U3 BQ24210DQCT

Commit message: Notecarrier-A v2.3: label the USB block USB-C, not Micro-USB
The Power sheet's block was still titled "Micro-USB", inherited from the v2.0
port it was scaffolded from. v2.3's whole point on that block is the opposite:
J11 is the Amphenol 12402012E212A USB-C receptacle, with the R32/R33 CC
pull-downs beside it, and the design house's own change list reads "Swap the
micro-USB to USB-C".

Caught while reviewing a kicanvas render of the sheet for publication - a
USB-C connector sitting inside a box labelled Micro-USB is the kind of thing a
reader trusts over the part number. Graphical text only; the exported netlist is
identical before and after.

Co-Authored-By: Claude Fable 5 <noreply@anthropic.com>
Other:
- note added: "USB-C"
- note removed: "Micro-USB"
Changed lines of the file:
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@@
 		)
 	)
-	(text "Micro-USB"
+	(text "USB-C"
 		(exclude_from_sim no)
 		(at 19.05 203.2 0)
