File: Notecarrier-F/v1.3/KiCad_format/Notecarrier-F_Feather.kicad_sch (KiCad schematic)
At the start: 23 parts, among them J7 SM04B-SRSS-TB(LF)(SN), J8 SM04B-SRSS-TB(LF)(SN), SW3 CJS-1200TA, SW4 CJS-1200TA, U1 TXS0102DCUR, U4 TXS0102DCUR, U5 DGQ2788AEN-T1-GE4, U6 DGQ2788AEN-T1-GE4

Commit message: Upgrade the four original ports to KiCad 9; fix F v1.3 DRC; document F errata
Notecarrier-A v2.0, -B v2.1, -F v1.3 and -Pi v1.1 were authored in KiCad 7 and
are now upgraded in place (board 20221018 -> 20241229, schematics -> 20250114).
The upgrade is verified lossless on all four:

- every fabrication layer (copper, mask, paste, silk, Edge.Cuts) is
  geometrically identical before and after at 600 dpi, and drill files are
  textually identical;
- schematic netlists are unchanged - same components, same net partitions
  (A 99/114, B 62/87, F 110/166, Pi 46/95);
- kicanvas renders and the RAG extract both still pass.

Zones are NOT refilled - these ports depend on preserved fills.

Notecarrier-F: the board's 54 net-less 0.6 mm copper patches (footprint
weird-no-fill-via_Fv1.2) sit inside GND copper and are now assigned the GND net
they belong to. DRC goes from 171 errors to 0 with no change to any copper
geometry.

Notecarrier-F ERRATA.md (new): the power section does not match the shipped
board. U9 (AP2139AK-3.3 LDO) with C33/C34, and DS7 (STPS3H100U), are missing
from both schematic and board though they are in the Altium source, the released
BOM, the released pick-and-place, and the shipped copper/mask/paste. All six
diodes carry the wrong part and package: the released design uses FSV1045V in
TO277-3 (3 pads) for DS1/DS2/DS4/DS5 and STPS3H100U in SMB for DS3/DS6/DS7,
where the port has B360A-13-F in DO-214AC SMA (2 pads) throughout. The errata
records the exact wiring and coordinates needed to fix it. Flagged in the root
README and the port's README.

Also documented per port: the DRC exclusions recorded by KiCad 7 no longer
suppress anything, because KiCad 9 computes different marker keys. They are left
as the author's record and the remaining violations are explained in each
Porting-Notes - including evidence that A's J9 pad-vs-zone reports are
preserved-fill artifacts (its In1 plane matches the shipped GND film to within
0.9% of lit area), and that B's 4 error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
Parts:
- renumbered C3 to C10, C3 to C11, C3 to C12, C3 to C13, C3 to C14, C3 to C15, R3 to R10, R3 to R11, R3 to R12, R3 to R15, R3 to R16, R3 to R18

Commit message: Notecarrier-F: apply the v1.2 -> v1.3 schematic delta
The schematic sheets now describe v1.3. Every step was verified by re-exporting
the netlist and comparing against the intended result rather than by
inspection, and the final state is tabulated in ERRATA.md.

- Adds U9 (AP2139AK-3.3TRG1 LDO) with C33/C34, wired as the released schematic
  draws it: VIN and CE both on the DS5 anode node, VOUT on the new F_VIO rail,
  NC left open with a no-connect marker.
- Migrates the six F_VIO nodes off F_BAT (U4.7, C14.1, U1.3, C11.1, R11.2,
  R12.2), leaving F_BAT with only DS5's cathode and the Feather BAT pin. This is
  the substance of the revision: both level shifters previously took their
  Feather-side supply from raw battery voltage.
- Adds DS7 (STPS3H100U) as the Notecard USB input diode.
- Re-parts the six diodes: DS1/DS2/DS4/DS5 to the 3-pin FSV1045V in TO277-3,
  DS3/DS6 to STPS3H100U in SMB.
- Marks R11/R12 DNP rather than deleting them, matching how the released
  schematic strikes them through, and adds a power_F_VIO symbol to the
  project-local library.

Three things did not go as the plan assumed, and the plan was wrong rather than
the files:

- The F_BAT net is four separate wire nodes unified by name, not one, and the
  node carrying C14.1/U4.7 was named by a plain local label sitting mid-wire
  that a hierarchical-label search does not see. Found by probing each naming
  object and re-exporting; no wire surgery turned out to be necessary.
- DS2 alone carries a lib_name override pinning it to a cached 2-pin symbol, so
  changing its lib_id silently did nothing. The netlist check caught it; every
  other diode was fine.
- MODL1/MODR1 cannot be renamed to the released MOD1L/MOD1R. KiCad takes the
  annotation number from a reference's trailing digits, so a name ending in a
  letter reads as unannotated and the exported BOM literally says "MOD1L?".
  Reverted, with the mapping to the released BOM documented instead.

The board still describes v1.2, so the sche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
Parts:
- R11, R12: now not fitted
Connections:
- net F_BAT: no longer C11.1, C14.1, R11.2, R12.2, U1.3 (VCCA), U4.7 (VCCB)
- new net F_VIO: C11.1, C14.1, R11.2, R12.2, U1.3 (VCCA), U4.7 (VCCB)
Changed lines of the file:
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@@
 		)
 	)
-	(label "F_BAT"
+	(label "F_VIO"
 		(at 74.93 119.38 0)
 		(effects
@@
 		)
 	)
-	(hierarchical_label "F_BAT"
-		(shape input)
-		(at 30.48 132.08 180)
-		(effects
-			(font
-				(size 1.27 1.27)
-			)
-			(justify right)
-		)
-	)
 	(hierarchical_label "F_EN"
 		(shape input)
@@
 	)
 	(symbol
+		(lib_id "Notecarrier-F-local:power_F_VIO")
+		(at 30.48 132.08 0)
+		(unit 1)
+		(exclude_from_sim no)
+		(in_bom no)
+		(on_board no)
+		(dnp no)
+		(property "Reference" "#PWR072"
+			(at 30.48 135.89 0)
+			(effects
+				(font
+					(size 1.27 1.27)
+				)
+				(hide yes)
+			)
+		)
+		(property "Value" "F_VIO"
+			(at 30.48 128.27 0)
+			(effects
+				(font
+					(size 1.27 1.27)
+				)
+			)
+		)
+		(property "Footprint" ""
+			(at 30.48 132.08 0)
+			(effects
+				(font
+					(size 1.27 1.27)
+				)
+				(hide yes)
+			)
+		)
+		(property "Datasheet" ""
+			(at 30.48 132.08 0)
+			(effects
+				(font
+					(size 1.27 1.27)
+				)
+				(hide yes)
+			)
+		)
+		(property "Description" ""
+			(at 30.48 132.08 0)
+			(effects
+				(font
+					(size 1.27 1.27)
+				)
+			)
+		)
+		(pin "1"
+		)
+		(instances
+			(project "Notecarrier-F"
+				(path "/3e57c059-f782-40ac-b9a3-c1636ed27a63/fb5887cf-5e51-4ae9-9749-dbe8e6b41d9d"
+					(reference "#PWR072")
+					(unit 1)
+				)
+			)
+		)
+	)
+	(symbol
 		(lib_id "power:GND")
 		(at 128.27 130.81 0)
@@
 	)
 	(symbol
-		(lib_id "blues-kicad-lib:power_F_BAT")
+		(lib_id "Notecarrier-F-local:power_F_VIO")
 		(at 144.78 92.71 0)
 		(unit 1)
@@
 			)
 		)
-		(property "Value" "F_BAT"
+		(property "Value" "F_VIO"
 			(at 144.78 88.9 0)
 			(effects
@@
 	)
 	(symbol
-		(lib_id "blues-kicad-lib:power_F_BAT")
+		(lib_id "Notecarrier-F-local:power_F_VIO")
 		(at 137.16 92.71 0)
 		(unit 1)
@@
 			)
 		)
-		(property "Value" "F_BAT"
+		(property "Value" "F_VIO"
 			(at 137.16 88.9 0)
 			(effects
@@
 		(in_bom yes)
 		(on_board yes)
-		(dnp no)
+		(dnp yes)
 		(property "Reference" "R12"
 			(at 149.86 96.52 0)
@@
 	)
 	(symbol
-		(lib_id "blues-kicad-lib:power_F_BAT")
+		(lib_id "Notecarrier-F-local:power_F_VIO")
 		(at 151.13 116.84 0)
 		(unit 1)
@@
 			)
 		)
-		(property "Value" "F_BAT"
+		(property "Value" "F_VIO"
 			(at 151.13 113.03 0)
 			(effects
@@
 		(in_bom yes)
 		(on_board yes)
-		(dnp no)
+		(dnp yes)
 		(property "Reference" "R11"
 			(at 142.24 96.52 0)

Commit message: Notecarrier-F: convert its design-note text_boxes too
The first conversion pass scoped by red-frame rectangles and missed
Notecarrier-F: its 16 notes have no separate frame - the text_box itself draws
a 0.5mm red border - so they were entirely invisible on the published pages,
frames included. Same conversion as 25a2d84, with two additions the F notes
forced:

- KiCad's hidden PDF text layer mangles special glyphs (broken ToUnicode maps
  for u/~/ohm produce mojibake) and F's notes are full of them, so exact
  word-matching is unattainable. Notes whose visual line count matches their
  source line count need no wrap-freezing at all and are kept verbatim, guarded
  by a per-line ASCII similarity check; only genuinely wrapped notes use the
  strict word-level path, and F's wrapped notes are clean of special glyphs.
  The converter also now rebuilds output from SOURCE words - the PDF only
  supplies break positions - so KiCad markup like R_{iset} stays markup in the
  file instead of being replaced by its rendered form.

- The F author gave these notes an explicit black font color. Black is what
  KiCad plots either way, but explicit black is invisible on a dark-theme
  viewer. The 16 notes now carry no explicit color, like every other board's
  notes: KiCad plots its default dark blue, kicanvas its theme color. This is
  the one deliberate visual change - note text black -> dark blue in KiCad -
  and it makes F consistent with the other five boards.

Netlist byte-equal before and after; kicanvas renders all four modified sheets
with the notes visible and the subscript markup intact.

Co-Authored-By: Claude Fable 5 <noreply@anthropic.com>
Other:
- note added: "DESIGN NOTE: - AUX SW"
- note added: "DESIGN NOTE: - FEATHER_EN SW"
- note added: "DESIGN NOTE: - OE is referenced to VCCA"
- note added: "SOFTWARE CONFIG NOTE: - Flick switch towards "ON" to enable outboard DFU"
- note added: "SOFTWARE CONFIG NOTE: Truth table: IN1-2, IN3-4 Logic 0 = NC is True/High, DFU = N Logic 1 = NO is True/High, DFU = Y"
Changed lines of the file:
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@@
 		)
 	)
-	(text_box "DESIGN NOTE:\n- AUX SW"
-		(exclude_from_sim no)
-		(at 50.8 72.39 0)
-		(size 21.59 6.35)
-		(margins 1.2025 1.2025 1.2025 1.2025)
+	(rectangle
+		(start 50.8 72.39)
+		(end 72.39 78.74)
 		(stroke
 			(width 0.5)
@@
 			(type none)
 		)
+	)
+	(text "DESIGN NOTE:\n- AUX SW"
+		(exclude_from_sim no)
+		(at 52.0025 73.5925 0)
 		(effects
 			(font
 				(size 1.27 1.27)
-				(color 0 0 0 1)
 			)
 			(justify left top)
 		)
 	)
-	(text_box "DESIGN NOTE:\n- OE is referenced to VCCA"
-		(exclude_from_sim no)
-		(at 171.45 125.73 0)
-		(size 30.48 6.35)
-		(margins 1.2025 1.2025 1.2025 1.2025)
+	(rectangle
+		(start 171.45 125.73)
+		(end 201.93 132.08)
 		(stroke
 			(width 0.5)
@@
 			(type none)
 		)
+	)
+	(text "DESIGN NOTE:\n- OE is referenced to VCCA"
+		(exclude_from_sim no)
+		(at 172.652 126.933 0)
 		(effects
 			(font
 				(size 1.27 1.27)
-				(color 0 0 0 1)
 			)
 			(justify left top)
 		)
 	)
-	(text_box "SOFTWARE CONFIG NOTE:\nTruth table:\nIN1-2, IN3-4\nLogic 0 = NC is True/High, DFU = N\nLogic 1 = NO is True/High, DFU = Y\n"
-		(exclude_from_sim no)
-		(at 38.1 41.91 0)
-		(size 40.64 12.7)
-		(margins 1.2025 1.2025 1.2025 1.2025)
+	(rectangle
+		(start 38.1 41.91)
+		(end 78.74 54.61)
 		(stroke
 			(width 0.5)
@@
 			(type none)
 		)
+	)
+	(text "SOFTWARE CONFIG NOTE:\nTruth table:\nIN1-2, IN3-4\nLogic 0 = NC is True/High, DFU = N\nLogic 1 = NO is True/High, DFU = Y\n"
+		(exclude_from_sim no)
+		(at 39.3025 43.1125 0)
 		(effects
 			(font
 				(size 1.27 1.27)
-				(color 0 0 0 1)
 			)
 			(justify left top)
 		)
 	)
-	(text_box "SOFTWARE CONFIG NOTE:\n- Flick switch towards \"ON\" to enable outboard DFU"
-		(exclude_from_sim no)
-		(at 38.1 26.67 0)
-		(size 40.64 12.7)
-		(margins 1.2025 1.2025 1.2025 1.2025)
+	(rectangle
+		(start 38.1 26.67)
+		(end 78.74 39.37)
 		(stroke
 			(width 0.5)
@@
 			(type none)
 		)
+	)
+	(text "SOFTWARE CONFIG NOTE:\n- Flick switch towards \"ON\" to enable\noutboard DFU"
+		(exclude_from_sim no)
+		(at 39.3025 27.8725 0)
 		(effects
 			(font
 				(size 1.27 1.27)
-				(color 0 0 0 1)
 			)
 			(justify left top)
 		)
 	)
-	(text_box "DESIGN NOTE:\n- FEATHER_EN SW"
-		(exclude_from_sim no)
-		(at 36.83 119.38 0)
-		(size 21.59 6.35)
-		(margins 1.2025 1.2025 1.2025 1.2025)
+	(rectangle
+		(start 36.83 119.38)
+		(end 58.42 125.73)
 		(stroke
 			(width 0.5)
@@
 			(type none)
 		)
+	)
+	(text "DESIGN NOTE:\n- FEATHER_EN SW"
+		(exclude_from_sim no)
+		(at 38.0325 120.582 0)
 		(effects
 			(font
 				(size 1.27 1.27)
-				(color 0 0 0 1)
 			)
 			(justify left top)
