File: Notecarrier-F/v1.3/KiCad_format/Notecarrier-F_Feather.kicad_sch (KiCad schematic)
At the start: 23 parts, among them J7 SM04B-SRSS-TB(LF)(SN), J8 SM04B-SRSS-TB(LF)(SN), SW3 CJS-1200TA, SW4 CJS-1200TA, U1 TXS0102DCUR, U4 TXS0102DCUR, U5 DGQ2788AEN-T1-GE4, U6 DGQ2788AEN-T1-GE4

Commit message: updated kicad files
Connections:
- net F_EN: no longer SW3.3 (A)
- net N_VIO: now also SW3.3 (A)
Changed lines of the file:
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@@
 	(wire
 		(pts
-			(xy 30.48 109.22) (xy 46.99 109.22)
-		)
-		(stroke
-			(width 0)
-			(type default)
-		)
-	)
-	(wire
-		(pts
 			(xy 190.5 36.83) (xy 207.01 36.83)
 		)
@@
 	(wire
 		(pts
-			(xy 30.48 149.86) (xy 78.74 149.86)
-		)
-		(stroke
-			(width 0)
-			(type default)
-		)
-	)
-	(wire
-		(pts
 			(xy 71.12 119.38) (xy 96.52 119.38)
 		)
@@
 		)
 	)
-	(label "F_EN"
-		(at 37.2695 109.22 0)
-		(effects
-			(font
-				(size 1.27 1.27)
-			)
-			(justify left bottom)
-		)
-	)
 	(label "SW_SCL"
 		(at 233.68 165.1 180)
@@
 		)
 	)
-	(hierarchical_label "F_NRST"
-		(shape input)
-		(at 30.48 149.86 180)
-		(effects
-			(font
-				(size 1.27 1.27)
-			)
-			(justify right)
-		)
-	)
 	(hierarchical_label "F_NRST_SW"
 		(shape input)
@@
 	(hierarchical_label "F_EN"
 		(shape input)
-		(at 30.48 109.22 180)
-		(effects
-			(font
-				(size 1.27 1.27)
-			)
-			(justify right)
-		)
-	)
-	(hierarchical_label "F_EN"
-		(shape input)
 		(at 154.94 162.56 0)
 		(effects
@@
 		)
 	)
-)
+	(wire
+		(pts
+			(xy 36.83 109.22) (xy 46.99 109.22)
+		)
+		(stroke
+			(width 0)
+			(type default)
+		)
+	)
+	(label "N_VIO"
+		(at 36.83 109.22 0)
+		(effects
+			(font
+				(size 1.27 1.27)
+			)
+			(justify left bottom)
+		)
+	)
+	(wire
+		(pts
+			(xy 36.83 149.86) (xy 78.74 149.86)
+		)
+		(stroke
+			(width 0)
+			(type default)
+		)
+	))
