File: Notecarrier-F/v1.3/KiCad_format/Notecarrier-F_Power-Input.kicad_sch (KiCad schematic)
At the start: 21 parts, among them J1 S2BPHSM4TBLFSN, J2 S2BPHSM4TBLFSN, J3 S2BPHSM4TBLFSN, J4 10118193-0001LF, U2 BQ24210DQCT

Commit message: updated kicad files
Parts:
- R3: value 499R -> 470R; Datasheet 2 https://datasheet.octopart.com/CR0402-FX-4990GLF-Bourns-dat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 -> (none); Datasheet 3 https://datasheet.octopart.com/RC0402FR-07499RP-Yageo-datas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 -> (none); Design Description Resistor 499R ±1% 0402 -> Resistor 470R ±1% 0402; Design MPN N/A -> RC0402FR-13470RL; Design Manufacturer N/A -> Yageo; MPN 0402WGF4990TCE -> RC0402FR-13470RL; MPN 2 CR0402-FX-4990GLF -> (none); MPN 3 RC0402FR-07499RP -> (none); Manufacturer Royal Ohm -> Yageo; Manufacturer 2 Bourns -> (none); Manufacturer 3 Yageo -> (none); Mfr Description Res Thick Film 0402 499 Ohm 1% 0.063W(1/16W) ±100ppm/°C Pad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 -> Resistor 470R ±1% 0402; Mfr Description 2 SMD Chip Resistor, 499 Ohm, ± 1%, 63 mW, 0402 [1005 Metric]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 -> (none); Mfr Description 3 Res General Purpose Thick Film 0402 499 Ohm 1% 1/16W ±100pp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 -> (none)
Other:
- note added: "DESIGN NOTE: - R_{iset} = K_{iset} / I_{out} - K_{iset} = 395 AΩ typically. - R_{iset} = 470R --> I_{out} = 800mA (v1.3; v1.2 used 499R / 791mA)"
- note removed: "DESIGN NOTE: - R_{iset} = K_{iset} / I_{out} - K_{iset} = 395 AΩ typically. - R_{iset} = 499R --> I_{out} = 791mA"
Changed lines of the file:
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@@
 		)
 	)
-	(text "DESIGN NOTE:\n- R_{iset} = K_{iset} / I_{out}\n- K_{iset} = 395 AΩ typically.\n- R_{iset} = 499R --> I_{out} = 791mA"
+	(text "DESIGN NOTE:\n- R_{iset} = K_{iset} / I_{out}\n- K_{iset} = 395 AΩ typically.\n- R_{iset} = 470R --> I_{out} = 800mA (v1.3; v1.2 used 499R / 791mA)"
 		(exclude_from_sim no)
 		(at 79.9425 77.4025 0)
@@
 			)
 		)
-		(property "Value" "499R"
+		(property "Value" "470R"
 			(at 58.42 76.2 0)
 			(effects
@@
 			)
 		)
-		(property "Datasheet" "https://datasheet.octopart.com/0402WGF4990TCE-Royal-Ohm-datasheet-165785611.pdf"
+		(property "Datasheet" "https://www.yageo.com/upload/media/product/productsearch/datasheet/rchip/PYu-RC_Group_51_RoHS_L_12.pdf"
 			(at 57.15 74.93 0)
 			(effects
@@
 			)
 		)
-		(property "Description" "RES 499 OHM 1% 1/16W SMT 0402"
+		(property "Description" "RES 470 OHM 1% 1/16W SMT 0402"
 			(at 57.15 74.93 0)
 			(effects
@@
 			)
 		)
-		(property "Manufacturer" "Royal Ohm"
+		(property "Manufacturer" "Yageo"
 			(at 57.15 74.93 0)
 			(effects
@@
 			)
 		)
-		(property "Datasheet 2" "https://datasheet.octopart.com/CR0402-FX-4990GLF-Bourns-datasheet-159578630.pdf"
+		(property "Datasheet 2" ""
 			(at 57.15 74.93 0)
 			(effects
@@
 			)
 		)
-		(property "Datasheet 3" "https://datasheet.octopart.com/RC0402FR-07499RP-Yageo-datasheet-164759695.pdf"
+		(property "Datasheet 3" ""
 			(at 57.15 74.93 0)
 			(effects
@@
 			)
 		)
-		(property "MPN" "0402WGF4990TCE"
+		(property "MPN" "RC0402FR-13470RL"
 			(at 57.15 74.93 0)
 			(effects
@@
 			)
 		)
-		(property "MPN 2" "CR0402-FX-4990GLF"
+		(property "MPN 2" ""
 			(at 57.15 74.93 0)
 			(effects
@@
 			)
 		)
-		(property "MPN 3" "RC0402FR-07499RP"
+		(property "MPN 3" ""
 			(at 57.15 74.93 0)
 			(effects
@@
 			)
 		)
-		(property "Manufacturer 2" "Bourns"
+		(property "Manufacturer 2" ""
 			(at 57.15 74.93 0)
 			(effects
@@
 			)
 		)
-		(property "Manufacturer 3" "Yageo"
+		(property "Manufacturer 3" ""
 			(at 57.15 74.93 0)
 			(effects
@@
 			)
 		)
-		(property "Mfr Description" "Res Thick Film 0402 499 Ohm 1% 0.063W(1/16W) ±100ppm/°C Pad SMD T/R"
+		(property "Mfr Description" "Resistor 470R ±1% 0402"
 			(at 57.15 74.93 0)
 			(effects
@@
 			)
 		)
-		(property "Mfr Description 2" "SMD Chip Resistor, 499 Ohm, ± 1%, 63 mW, 0402 [1005 Metric], Thick Film, General Purpose"
+		(property "Mfr Description 2" ""
 			(at 57.15 74.93 0)
 			(effects
@@
 			)
 		)
-		(property "Mfr Description 3" "Res General Purpose Thick Film 0402 499 Ohm 1% 1/16W ±100ppm/°C Molded SMD Paper T/R"
+		(property "Mfr Description 3" ""
 			(at 57.15 74.93 0)
 			(effects
@@
 			)
 		)
-		(property "Design Description" "Resistor 499R ±1% 0402"
+		(property "Design Description" "Resistor 470R ±1% 0402"
 			(at 57.15 74.93 0)
 			(effects
@@
 			)
 		)
-		(property "Design MPN" "N/A"
+		(property "Design MPN" "RC0402FR-13470RL"
 			(at 57.15 74.93 0)
 			(effects
@@
 			)
 		)
-		(property "Design Manufacturer" "N/A"
+		(property "Design Manufacturer" "Yageo"
 			(at 57.15 74.93 0)
 			(effects
