File: Notecarrier-XM/v1.2/KiCad_format/Notecarrier-XM.kicad_pcb (KiCad board)
At the start: 2 copper layers, 57.1 x 38.1 mm, 26 parts, among them J5 MDT420E01001, P1 Header Castellated 2.54mm 1X16, P2 Header Castellated 2.54mm 1X16, P3 12402012E212A, U1 ISL9122AIINZ-T, U3 LM66200DRLR

Commit message: feat: updates to X, XM, XS Notecarrier files (#49)
* Notecarrier-X/XM: add board-regeneration scripts

Scripts used to regenerate the X and XM v1.2 boards from the design
house's Rev-11 release snapshots while keeping everything else in the
published ports:

- sanitize_fonts.py: zero the padding after each Texts6 font name in a
  copy of the PcbDoc. KiCad 9.0.9's Altium importer converts the whole
  64-byte UTF-16 field, and leftover bytes containing an unpaired
  surrogate make it drop the TrueType face (and size the text as
  stroke text).
- pcb_import.py: headless PcbDoc -> .kicad_pcb import.
- transplant.py: swap the Rev-11 tracks, vias, zones (original fills)
  and board graphics into the published port's file, renumbering nets
  by name through pad correspondence; 3-way merge for the moved jumper.

Co-Authored-By: Claude Opus 5.5 <noreply@anthropic.com>

* Notecarrier-X v1.2: regenerate board from the Rev-11 release snapshot

The port was first built from a post-v1.2 development state and carried
a source-fidelity disclaimer (silk read V1.3; the production-DNP jumper
R4 sat on the bottom side). The design house has now supplied the Rev-11
snapshot behind the published v1.2 fab package (2200-918, 3000-794-001).

- Schematic unchanged: the Rev-11 electrical sheets are identical in
  substance to the development state (template differences only).
- Board regenerated from Rev-11: R4 back on top with its local routing,
  re-poured GND fills, silk V1.2 / RST. Footprints, schematic links,
  BOM fields, rules and project settings carried over unchanged.
- Verified: all harness gates pass; copper/mask/paste 0.001-0.010 vs the
  published fab with no difference cluster >= 0.045 mm2 (baseline
  tightened); every pad's net matches the Rev-11 board
  (validation/altium-netlist-compare.txt, 0 conflicts, 56 nets).
- Fab zip and layer PDF re-exported; Porting-Notes and READMEs updated,
  disclaimer retired.

Co-Authored-By: Claude Opus 5.5 <noreply@anthropic.com>

* Notecarri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
Parts:
- moved R2 33.7 mm to (146.6, 118.0), turned to 90 degrees
Routing:
- net +VACT_GPS_OUT: track 57.7 -> 20.6 mm, vias 6 -> 2
- net +VACT_GPS_IN: track 55.7 -> 21.5 mm, vias 6 -> 2
- net AUX_NCHARGING: track 26.1 -> 24.1 mm
- net +VMAIN: track 59.2 -> 57.6 mm
- net GND: track 38.8 -> 37.6 mm, vias 176 -> 180
Other:
- board text added: "226"
- board text added: "303 Total"
- board text added: "RST"
- board text removed: "230"
- board text removed: "307 Total"
- board text removed: "VGPS"
